File: hardware/pumpengruppe-rs485/pumpengruppe-rs485.kicad_pcb (KiCad board)
At the start: 2 copper layers, 160 x 110 mm, 111 parts, among them J1 RJ45_IN, J2 RJ45_OUT, J3 RS485_IN, J4 RS485_OUT, K1 PUMP_RELAY, K2 MIX_ENABLE_RELAY, K3 MIX_DIR_SPDT_RELAY, Q1 AO3400A_PUMP, Q2 AO3400A_MIX_ENABLE, Q3 AO3400A_MIX_DIR, U1 ESP32-WROOM-32D, U2 MAX31865_VL, U3 MAX31865_RL, U4 MAX3485_SOIC8, U5 3V3_REG, U6 CP2102N_USB_UART, X1 230V_IN, X2 PUMPE, X3 MISCHER, X4 RTD_VL, X5 RTD_RL, X6 USB_C_SERVICE_FLASH

Commit message: icherung
Routing:
- net GND: track 628.2 -> 647.0 mm, vias 10 -> 12
- net +3V3: track 161.7 -> 178.5 mm, vias 0 -> 2
- net RGB_DOUT_15: track 0.00 -> 12.6 mm, vias 0 -> 2
- net +5V: track 519.0 -> 524.6 mm

Commit message: sicherung
Parts:
- added MB1: BREAKAWAY_MOUSEBITES, FW_Pumpengruppe:BREAKAWAY_MOUSEBITES, F.Cu at (84.0, 0.00)
Routing:
- net +5V: track 524.6 -> 748.9 mm, vias 6 -> 7
- net GND: track 647.0 -> 844.1 mm, vias 12 -> 13
- net RS485_GND: track 117.3 -> 176.2 mm
- net BUS_5V: track 36.5 -> 62.6 mm, vias 0 -> 2
- net USB_VBUS: track 71.7 -> 76.5 mm, vias 0 -> 2
- net RGB_DOUT_15: track 12.6 -> 8.00 mm, vias 2 -> 0
- net +3V3: track 178.5 -> 182.9 mm
- net RS485_B: track 138.0 -> 140.7 mm
- net USB_CC1: track 21.3 -> 21.2 mm, vias 0 -> 2
Other:
- board text added: "DNP IN TEMP VARIANT"
- board text added: "POWER VIA RJ45 BUS_5V"
- board text added: "TEMP INPUT: LEFT 230V/RELAY SIDE DNP"

Commit message: sicherung
Parts:
- C60, C61, C62, C63, C64, C65, C66, C67, C68, C69, C70, C71, C72, C73, C74, C75, C76, C77, C78, C79, C80, C81, C82, C83: value 100n_RGB_LED -> 100nF 16V
- D1: value SS14_FLYBACK_PUMP -> B5819W; footprint FW_Pumpengruppe:D_SOD123 -> Diode_SMD:D_SOD-123
- D10: value LED_PUMP -> LED green 0603; footprint FW_Pumpengruppe:LED_0603 -> LED_SMD:LED_0603_1608Metric
- D11: value LED_MIX_ENABLE -> LED green 0603; footprint FW_Pumpengruppe:LED_0603 -> LED_SMD:LED_0603_1608Metric
- D12: value LED_MIX_DIR -> LED green 0603; footprint FW_Pumpengruppe:LED_0603 -> LED_SMD:LED_0603_1608Metric
- D2: value SS14_FLYBACK_MIX_ENABLE -> B5819W; footprint FW_Pumpengruppe:D_SOD123 -> Diode_SMD:D_SOD-123
- D20: value LED_5V -> LED green 0603; footprint FW_Pumpengruppe:LED_0603 -> LED_SMD:LED_0603_1608Metric
- D21: value LED_3V3 -> LED green 0603; footprint FW_Pumpengruppe:LED_0603 -> LED_SMD:LED_0603_1608Metric
- D3: value SS14_FLYBACK_MIX_DIR -> B5819W; footprint FW_Pumpengruppe:D_SOD123 -> Diode_SMD:D_SOD-123
- D30: value LED_RS485_TX -> LED green 0603; footprint FW_Pumpengruppe:LED_0603 -> LED_SMD:LED_0603_1608Metric
- D31: value LED_RS485_RX -> LED green 0603; footprint FW_Pumpengruppe:LED_0603 -> LED_SMD:LED_0603_1608Metric
- D4: value SS14_USB_TO_5V -> B5819W; footprint FW_Pumpengruppe:D_SOD123 -> Diode_SMD:D_SOD-123
- D40: value LED_230VAC -> LED green 0805
- D41: value 1N4148_ANTI_PARALLEL -> 1N4148W
- D50: value TVS_RS485_A_COM -> DNP TVS SOD-123
- D51: value TVS_RS485_B_COM -> DNP TVS SOD-123
- D52: value TVS_RS485_A_B -> DNP TVS SOD-123
- D60: value SK6812MINI_STATUS_1 -> SK6812MINI-E
- D61: value SK6812MINI_STATUS_2 -> SK6812MINI-E
- D62: value SK6812MINI_STATUS_3 -> SK6812MINI-E
- D63: value SK6812MINI_STATUS_4 -> SK6812MINI-E
- D64: value SK6812MINI_VALVE_5PCT -> SK6812MINI-E
- D65: value SK6812MINI_VALVE_10PCT -> SK6812MINI-E
- D66: value SK6812MINI_VALVE_15PCT -> SK6812MINI-E
- D67: value SK6812MINI_VALVE_20PCT -> SK6812MINI-E
- D68: value SK6812MINI_VALVE_25PCT -> SK6812MINI-E
- D69: value SK6812MINI_VALVE_30PCT -> SK6812MINI-E
- D70: value SK6812MINI_VALVE_35PCT -> SK6812MINI-E
- D71: value SK6812MINI_VALVE_40PCT -> SK6812MINI-E
- D72: value SK6812MINI_VALVE_45PCT -> SK6812MINI-E
- D73: value SK6812MINI_VALVE_50PCT -> SK6812MINI-E
- D74: value SK6812MINI_VALVE_55PCT -> SK6812MINI-E
- D75: value SK6812MINI_VALVE_60PCT -> SK6812MINI-E
- D76: value SK6812MINI_VALVE_65PCT -> SK6812MINI-E
- D77: value SK6812MINI_VALVE_70PCT -> SK6812MINI-E
- D78: value SK6812MINI_VALVE_75PCT -> SK6812MINI-E
- D79: value SK6812MINI_VALVE_80PCT -> SK6812MINI-E
- D80: value SK6812MINI_VALVE_85PCT -> SK6812MINI-E
- D81: value SK6812MINI_VALVE_90PCT -> SK6812MINI-E
- D82: value SK6812MINI_VALVE_95PCT -> SK6812MINI-E
- D83: value SK6812MINI_VALVE_100PCT -> SK6812MINI-E
- F1: value TBD_T2A_T4A -> 5x20 fuse holder
- F2: value PTC_BUS_5V -> PTC 1.1A 1812
- J1: value RJ45_IN -> RJ45 8P8C horizontal
- J2: value RJ45_OUT -> RJ45 8P8C horizontal
- J3: value RS485_IN -> 3-pin 3.5mm terminal
- J4: value RS485_OUT -> 3-pin 3.5mm terminal
- JP1: value RS485_TERM_ON_PARK -> 1x3 2.54mm header
- K1: value PUMP_RELAY -> G5LE-1A-E DC5
- K2: value MIX_ENABLE_RELAY -> G5LE-1A-E DC5
- K3: value MIX_DIR_SPDT_RELAY -> G5LE-1 DC5
- PSU1: value HLK-5M05 -> IRM-05-5; footprint Converter_ACDC:Converter_ACDC_Hi-Link_HLK-5Mxx -> Converter_ACDC:Converter_ACDC_MeanWell_IRM-05-xx_THT
- Q1: value AO3400A_PUMP -> AO3400A; footprint FW_Pumpengruppe:SOT23_NMOS -> Package_TO_SOT_SMD:SOT-23
- Q2: value AO3400A_MIX_ENABLE -> AO3400A; footprint FW_Pumpengruppe:SOT23_NMOS -> Package_TO_SOT_SMD:SOT-23
- Q3: value AO3400A_MIX_DIR -> AO3400A; footprint FW_Pumpengruppe:SOT23_NMOS -> Package_TO_SOT_SMD:SOT-23
- R1: value 5k1_CC1 -> 5.1k 1% 0603; footprint FW_Pumpengruppe:R_0603 -> Resistor_SMD:R_0603_1608Metric
- R10: value 2k2_LED_PUMP -> 2.2k 1% 0603; footprint FW_Pumpengruppe:R_0603 -> Resistor_SMD:R_0603_1608Metric
- R11: value 2k2_LED_MIX_ENABLE -> 2.2k 1% 0603; footprint FW_Pumpengruppe:R_0603 -> Resistor_SMD:R_0603_1608Metric
- R12: value 2k2_LED_MIX_DIR -> 2.2k 1% 0603; footprint FW_Pumpengruppe:R_0603 -> Resistor_SMD:R_0603_1608Metric
- R2: value 5k1_CC2 -> 5.1k 1% 0603; footprint FW_Pumpengruppe:R_0603 -> Resistor_SMD:R_0603_1608Metric
- R20: value 2k2_LED_5V -> 2.2k 1% 0603; footprint FW_Pumpengruppe:R_0603 -> Resistor_SMD:R_0603_1608Metric
- R21: value 1k5_LED_3V3 -> 1.5k 1% 0603; footprint FW_Pumpengruppe:R_0603 -> Resistor_SMD:R_0603_1608Metric
- R3: value 120R_RS485_TERM -> 120R 1% 0603; footprint FW_Pumpengruppe:R_0603 -> Resistor_SMD:R_0603_1608Metric
- R30: value 4k7_LED_TX -> 4.7k 1% 0603; footprint FW_Pumpengruppe:R_0603 -> Resistor_SMD:R_0603_1608Metric
- R31: value 4k7_LED_RX -> 4.7k 1% 0603; footprint FW_Pumpengruppe:R_0603 -> Resistor_SMD:R_0603_1608Metric
- R32: value 0R_BUS_0V_LINK -> 0R 0603; footprint FW_Pumpengruppe:R_0603 -> Resistor_SMD:R_0603_1608Metric
- R4: value 100R_GATE_PUMP -> 100R 1% 0603; footprint FW_Pumpengruppe:R_0603 -> Resistor_SMD:R_0603_1608Metric
- R40: value 150k_LED_230V_1 -> 150k 1% 1206
- R41: value 150k_LED_230V_2 -> 150k 1% 1206
- R5: value 100R_GATE_MIX_ENABLE -> 100R 1% 0603; footprint FW_Pumpengruppe:R_0603 -> Resistor_SMD:R_0603_1608Metric
- R6: value 100R_GATE_MIX_DIR -> 100R 1% 0603; footprint FW_Pumpengruppe:R_0603 -> Resistor_SMD:R_0603_1608Metric
- R60: value 330R_RGB_DATA -> 330R 1% 0603
- R7, R8, R9: value 100k_GATE_PD -> 100k 1% 0603; footprint FW_Pumpengruppe:R_0603 -> Resistor_SMD:R_0603_1608Metric
- RV1: value MOV_275VAC -> MOV 275VAC
- U1: value ESP32-WROOM-32D -> ESP32-WROOM-32D-N4
- U2: value MAX31865_VL -> MAX31865AAP+; footprint FW_Pumpengruppe:SOIC16_RTD -> Package_SO:SOIC-16_3.9x9.9mm_P1.27mm
- U3: value MAX31865_RL -> MAX31865AAP+; footprint FW_Pumpengruppe:SOIC16_RTD -> Package_SO:SOIC-16_3.9x9.9mm_P1.27mm
- U4: value MAX3485_SOIC8 -> MAX3485EESA+
- U5: value 3V3_REG -> AMS1117-3.3; footprint FW_Pumpengruppe:LDO_SOT223 -> Package_TO_SOT_SMD:SOT-223-3_TabPin2
- U6: value CP2102N_USB_UART -> CP2102N-A02-GQFN24; footprint FW_Pumpengruppe:USB_UART_QFN24 -> Package_DFN_QFN:QFN-24-1EP_4x4mm_P0.5mm_EP2.7x2.7mm
- X1: value 230V_IN -> 3-pin 7.62mm terminal
- X2: value PUMPE -> 3-pin 7.62mm terminal
- X3: value MISCHER -> 4-pin 7.62mm terminal
- X4: value RTD_VL -> 2-pin 3.5mm terminal
- X5: value RTD_RL -> 2-pin 3.5mm terminal
- X6: value USB_C_SERVICE_FLASH -> USB-C receptacle
- moved R3 15.0 mm to (171.5, 102.0)
- moved PSU1 14.0 mm to (64.0, 58.0)
- moved J1 10.5 mm to (188.7, 84.2)
- moved J2 10.5 mm to (188.7, 101.2)
- moved F2 9.51 mm to (171.0, 88.5)
- moved JP1 9.01 mm to (176.0, 96.5)
Connections:
- PSU1 pad 3: +5V -> GND
- PSU1 pad 4: GND -> +5V
Routing:
- net RS485_GND: track 176.2 -> 106.7 mm
- net GND: track 844.1 -> 794.3 mm
- net +5V: track 748.9 -> 776.1 mm, vias 7 -> 6
- net RS485_A: track 138.1 -> 118.1 mm, vias 0 -> 2
- net BUS_5V: track 62.6 -> 44.7 mm, vias 2 -> 1
- net UART_TX: track 186.6 -> 200.0 mm
- net RS485_B: track 140.7 -> 130.0 mm
- net L_FUSED: track 91.7 -> 96.0 mm
- net RS485_TERM: track 3.75 -> 6.53 mm
- net N: track 138.9 -> 141.5 mm
