File: hardware/pumpengruppe-rs485/pumpengruppe-rs485.kicad_pcb (KiCad board)
At the start: 2 copper layers, 160 x 110 mm, 112 parts, among them J1 RJ45 8P8C horizontal, J2 RJ45 8P8C horizontal, J3 3-pin 3.5mm terminal, J4 3-pin 3.5mm terminal, K1 G5LE-1A-E DC5, K2 G5LE-1A-E DC5, K3 G5LE-1 DC5, Q1 AO3400A, Q2 AO3400A, Q3 AO3400A, U1 ESP32-WROOM-32D-N4, U2 MAX31865AAP+, U3 MAX31865AAP+, U4 MAX3485EESA+, U5 AMS1117-3.3, U6 CP2102N-A02-GQFN24, X1 3-pin 7.62mm terminal, X2 3-pin 7.62mm terminal, X3 4-pin 7.62mm terminal, X4 2-pin 3.5mm terminal, X5 2-pin 3.5mm terminal, X6 USB-C receptacle

Commit message: sicherung
Parts:
- added C22: 10nF 50V, Capacitor_SMD:C_0603_1608Metric, F.Cu at (180.6, 35.3)
- added C23: 10nF 50V, Capacitor_SMD:C_0603_1608Metric, F.Cu at (180.3, 58.8)
- added R22: 4.3k 0.1% 0603, Resistor_SMD:R_0603_1608Metric, F.Cu at (187.9, 41.8)
- added R23: 4.3k 0.1% 0603, Resistor_SMD:R_0603_1608Metric, F.Cu at (188.4, 51.2)
- added R33: 10k 1% 0603, Resistor_SMD:R_0603_1608Metric, F.Cu at (148.5, 36.8)
- F1: footprint FW_Pumpengruppe:FUSE_5X20 -> Fuse:Fuseholder_Clip-5x20mm_Bel_FC-203-22_Lateral_P17.80x5.00mm_D1.17mm_Horizontal
- U2, U3: footprint Package_SO:SOIC-16_3.9x9.9mm_P1.27mm -> Package_SO:SSOP-20_5.3x7.2mm_P0.65mm
- U6: footprint Package_DFN_QFN:QFN-24-1EP_4x4mm_P0.5mm_EP2.7x2.7mm -> Package_DFN_QFN:QFN-24-1EP_4x4mm_P0.5mm_EP2.6x2.6mm
- moved D4 11.4 mm to (134.0, 135.8)
- moved F1 10.7 mm to (63.0, 77.6)
- moved D20 7.58 mm to (174.8, 75.4)
- moved D21 6.94 mm to (174.9, 80.2)
- moved R21 6.13 mm to (169.7, 80.1)
- moved R20 6.08 mm to (169.8, 75.5)
- moved JP1 2.40 mm to (176.1, 98.9), turned to 180 degrees
- moved D12 0.15 mm to (106.9, 133.0)
Connections:
- net +5V renamed /+5V
- net BUS_5V renamed /BUS_5V
- net LED230_A renamed /MAINS_LED_K
- net LED230_DROP renamed /MAINS_LED_SERIES
- net LED_3V3_A renamed /LED_3V3_K
- net LED_5V_A renamed /LED_5V_K
- net LED_CLOSE_A renamed /LED_MIX_DIR_K
- net LED_OPEN_A renamed /LED_MIX_ENABLE_K
- net LED_PUMP_A renamed /LED_PUMP_K
- net LED_RX_A renamed /LED_USB_RX_K
- net LED_TX_A renamed /LED_USB_TX_K
- net L_CLOSE renamed /L_MIX_CLOSE
- net L_FUSED renamed /L_FUSED
- net L_IN renamed /L_IN
- net L_OPEN renamed /L_MIX_OPEN
- net L_PUMP renamed /L_PUMP
- net MIX_DIR_COIL_L renamed /MIX_DIR_COIL_DRV
- net MIX_DIR_DRV renamed /MIX_DIR_DRV_GPIO
- net MIX_DIR_GATE renamed /MIX_DIR_DRV
- net MIX_ENABLE_COIL_L renamed /MIX_ENABLE_COIL_DRV
- net MIX_ENABLE_DRV renamed /MIX_ENABLE_DRV_GPIO
- net MIX_ENABLE_GATE renamed /MIX_ENABLE_DRV
- net MIX_L_EN renamed /L_MIX_ENABLE
- net PUMP_COIL_L renamed /PUMP_COIL_DRV
- net PUMP_DRV renamed /PUMP_DRV_GPIO
- net PUMP_GATE renamed /PUMP_DRV
- net RGB_DATA renamed /RGB_DATA
- net RGB_DIN_1 renamed /RGB_D60_DIN
- net RGB_DOUT_1 renamed /RGB_D60_DOUT
- net RGB_DOUT_10 renamed /RGB_D69_DOUT
- net RGB_DOUT_11 renamed /RGB_D70_DOUT
- net RGB_DOUT_12 renamed /RGB_D71_DOUT
- net RGB_DOUT_13 renamed /RGB_D72_DOUT
- net RGB_DOUT_14 renamed /RGB_D73_DOUT
- net RGB_DOUT_15 renamed /RGB_D74_DOUT
- net RGB_DOUT_16 renamed /RGB_D75_DOUT
- net RGB_DOUT_17 renamed /RGB_D76_DOUT
- net RGB_DOUT_18 renamed /RGB_D77_DOUT
- net RGB_DOUT_19 renamed /RGB_D78_DOUT
- net RGB_DOUT_2 renamed /RGB_D61_DOUT
- net RGB_DOUT_20 renamed /RGB_D79_DOUT
- net RGB_DOUT_21 renamed /RGB_D80_DOUT
- net RGB_DOUT_22 renamed /RGB_D81_DOUT
- net RGB_DOUT_23 renamed /RGB_D82_DOUT
- net RGB_DOUT_3 renamed /RGB_D62_DOUT
- net RGB_DOUT_4 renamed /RGB_D63_DOUT
- net RGB_DOUT_5 renamed /RGB_D64_DOUT
- net RGB_DOUT_6 renamed /RGB_D65_DOUT
- net RGB_DOUT_7 renamed /RGB_D66_DOUT
- net RGB_DOUT_8 renamed /RGB_D67_DOUT
- net RGB_DOUT_9 renamed /RGB_D68_DOUT
- net RS485_A renamed /RS485_A
- net RS485_B renamed /RS485_B
- net RS485_DE renamed /RS485_DE
- net RS485_GND renamed /RS485_GND
- net RS485_TERM renamed /RS485_TERM
- net USB_CC1 renamed /USB_CC1
- net USB_CC2 renamed /USB_CC2
- C60 pad 2: GND -> /GND
- C61 pad 2: GND -> /GND
- C62 pad 2: GND -> /GND
- C63 pad 2: GND -> /GND
- C64 pad 2: GND -> /GND
- C65 pad 2: GND -> /GND
- C66 pad 2: GND -> /GND
- C67 pad 2: GND -> /GND
- C68 pad 2: GND -> /GND
- C69 pad 2: GND -> /GND
- C70 pad 2: GND -> /GND
- C71 pad 2: GND -> /GND
- C72 pad 2: GND -> /GND
- C73 pad 2: GND -> /GND
- C74 pad 2: GND -> /GND
- C75 pad 2: GND -> /GND
- C76 pad 2: GND -> /GND
- C77 pad 2: GND -> /GND
- C78 pad 2: GND -> /GND
- C79 pad 2: GND -> /GND
- C80 pad 2: GND -> /GND
- C81 pad 2: GND -> /GND
- C82 pad 2: GND -> /GND
- C83 pad 2: GND -> /GND
- D20 pad 2: GND -> /GND
- D21 pad 2: GND -> /GND
- D30 pad 2: UART_TX -> /ESP_U0TX
- D31 pad 2: UART_RX -> /ESP_U0RX
- D4 pad 2: USB_VBUS -> /USB_VBUS
- D40 pad 2: N -> /N
- D41 pad 1: N -> /N
- D60 pad 2: GND -> /GND
- D61 pad 2: GND -> /GND
- D62 pad 2: GND -> /GND
- D63 pad 2: GND -> /GND
- D64 pad 2: GND -> /GND
- D65 pad 2: GND -> /GND
- D66 pad 2: GND -> /GND
- D67 pad 2: GND -> /GND
- D68 pad 2: GND -> /GND
- D69 pad 2: GND -> /GND
- D70 pad 2: GND -> /GND
- D71 pad 2: GND -> /GND
- D72 pad 2: GND -> /GND
- D73 pad 2: GND -> /GND
- D74 pad 2: GND -> /GND
- D75 pad 2: GND -> /GND
- D76 pad 2: GND -> /GND
- D77 pad 2: GND -> /GND
- D78 pad 2: GND -> /GND
- D79 pad 2: GND -> /GND
- D80 pad 2: GND -> /GND
- D81 pad 2: GND -> /GND
- D82 pad 2: GND -> /GND
- D83 pad 1: RGB_DOUT_24 -> unconnected-(D83-DOUT-Pad1)
- D83 pad 2: GND -> /GND
- J1 pad 3: (no net) -> unconnected-(J1-Pin_3-Pad3)
- J1 pad 6: (no net) -> unconnected-(J1-Pin_6-Pad6)
- J2 pad 3: (no net) -> unconnected-(J2-Pin_3-Pad3)
- J2 pad 6: (no net) -> unconnected-(J2-Pin_6-Pad6)
- JP1 pad 3: (no net) -> unconnected-(JP1-Pin_3-Pad3)
- PSU1 pad 2: N -> /N
- PSU1 pad 3: GND -> /GND
- Q1 pad 2: GND -> /GND
- Q2 pad 2: GND -> /GND
- Q3 pad 2: GND -> /GND
- R1 pad 2: GND -> /GND
- R2 pad 2: GND -> /GND
- R21 pad 1: +3V3 -> /+3V3
- R30 pad 1: +3V3 -> /+3V3
- R31 pad 1: +3V3 -> /+3V3
- R32 pad 2: GND -> /GND
- R7 pad 2: GND -> /GND
- R8 pad 2: GND -> /GND
- R9 pad 2: GND -> /GND
- RV1 pad 2: N -> /N
- U1 pad 1: GND -> /GND
- U1 pad 13: (no net) -> unconnected-(U1-IO14-Pad13)
- U1 pad 14: (no net) -> unconnected-(U1-IO12-Pad14)
- U1 pad 15: GND -> /GND
- U1 pad 16: (no net) -> unconnected-(U1-IO13-Pad16)
- U1 pad 17: (no net) -> unconnected-(U1-SHD/SD2-Pad17)
- U1 pad 18: (no net) -> unconnected-(U1-SWP/SD3-Pad18)
- U1 pad 19: (no net) -> unconnected-(U1-SCS/CMD-Pad19)
- U1 pad 2: +3V3 -> /+3V3
- U1 pad 20: (no net) -> unconnected-(U1-SCK/CLK-Pad20)
- U1 pad 21: (no net) -> unconnected-(U1-SDO/SD0-Pad21)
- U1 pad 22: (no net) -> unconnected-(U1-SDI/SD1-Pad22)
- U1 pad 23: (no net) -> unconnected-(U1-IO15-Pad23)
- U1 pad 24: (no net) -> unconnected-(U1-IO2-Pad24)
- U1 pad 25: (no net) -> unconnected-(U1-IO0-Pad25)
- U1 pad 27: (no net) -> /RS485_UART_RX
- U1 pad 28: (no net) -> /RS485_UART_TX
- U1 pad 29: (no net) -> /RTD_VL_CS
- U1 pad 3: (no net) -> /ESP_EN
- U1 pad 30: SPI_SCK -> /SPI_SCK
- U1 pad 31: SPI_MISO -> /SPI_MISO
- U1 pad 32: (no net) -> unconnected-(U1-NC-Pad32)
- U1 pad 34: UART_RX -> /ESP_U0RX
- U1 pad 35: UART_TX -> /ESP_U0TX
- U1 pad 36: (no net) -> /RTD_RL_CS
- U1 pad 37: SPI_MOSI -> /SPI_MOSI
- U1 pad 38: GND -> /GND
- U1 pad 39: GND -> /GND
- U1 pad 4: (no net) -> unconnected-(U1-SENSOR_VP-Pad4)
- U1 pad 5: (no net) -> unconnected-(U1-SENSOR_VN-Pad5)
- U1 pad 6: (no net) -> unconnected-(U1-IO34-Pad6)
- U1 pad 7: (no net) -> unconnected-(U1-IO35-Pad7)
- U1 pad 8: (no net) -> unconnected-(U1-IO32-Pad8)
- U1 pad 9: (no net) -> unconnected-(U1-IO33-Pad9)
- U2 pad 1: RTD_VL_P -> unconnected-(U2-~{DRDY}-Pad1)
- U2 pad 10: SPI_MOSI -> /RTD_VL_FORCE_PLUS
- U2 pad 11: SPI_MISO -> /RTD_VL_FORCE_MINUS
- U2 pad 16: +3V3 -> /RTD_VL_CS
- U2 pad 2: RTD_VL_N -> /+3V3
- U2 pad 8: GND -> /RTD_VL_FORCE_PLUS
- U2 pad 9: SPI_SCK -> /RTD_VL_FORCE_PLUS
- U3 pad 1: RTD_RL_P -> unconnected-(U3-~{DRDY}-Pad1)
- U3 pad 10: SPI_MOSI -> /RTD_RL_FORCE_PLUS
- U3 pad 11: SPI_MISO -> /RTD_RL_FORCE_MINUS
- U3 pad 16: +3V3 -> /RTD_RL_CS
- U3 pad 2: RTD_RL_N -> /+3V3
- U3 pad 8: GND -> /RTD_RL_FORCE_PLUS
- U3 pad 9: SPI_SCK -> /RTD_RL_FORCE_PLUS
- U4 pad 1: UART_RX -> /RS485_UART_RX
- U4 pad 4: UART_TX -> /RS485_UART_TX
- U4 pad 5: GND -> /GND
- U4 pad 8: +3V3 -> /+3V3
- U5 pad 1: GND -> /GND
- U5 pad 2: +3V3 -> /+3V3
- U6 pad 1: USB_VBUS -> unconnected-(U6-~{RI}/CLK-Pad1)
- U6 pad 2: USB_D+ -> /GND
- U6 pad 3: USB_D- -> /USB_D+
- U6 pad 4: GND -> /USB_D-
- U6 pad 5: UART_RX -> /+3V3
- U6 pad 6: UART_TX -> /+3V3
- U6 pad 7: (no net) -> /USB_VBUS
- U6 pad 8: (no net) -> /USB_VBUS
- X1 pad 2: N -> /N
- X1 pad 3: PE -> /PE
- X2 pad 2: N -> /N
- X2 pad 3: PE -> /PE
- X3 pad 3: N -> /PE
- X3 pad 4: PE -> /N
- X4 pad 1: RTD_VL_P -> /RTD_VL_FORCE_PLUS
- X4 pad 2: RTD_VL_N -> /RTD_VL_FORCE_MINUS
- X5 pad 1: RTD_RL_P -> /RTD_RL_FORCE_PLUS
- X5 pad 2: RTD_RL_N -> /RTD_RL_FORCE_MINUS
- X6 pad A4: USB_VBUS -> /USB_VBUS
- X6 pad A6: USB_D+ -> /USB_D+
- X6 pad A7: USB_D- -> /USB_D-
- X6 pad A8: GND -> unconnected-(X6-SBU1-PadA8)
- X6 pad B4: USB_VBUS -> /USB_VBUS
- X6 pad B6: USB_D+ -> /USB_D+
- X6 pad B7: USB_D- -> /USB_D-
- X6 pad B8: GND -> unconnected-(X6-SBU2-PadB8)
- X6 pad SH: GND -> /GND
Routing:
- net GND: track 794.3 -> 0.00 mm, vias 13 -> 0
- net /GND: track 0.00 -> 720.0 mm, vias 0 -> 8
- net /+3V3: track 0.00 -> 256.0 mm, vias 0 -> 7
- net /+5V: track 776.1 -> 529.5 mm
- net UART_TX: track 200.0 -> 0.00 mm
- net +3V3: track 182.9 -> 0.00 mm, vias 2 -> 0
- net UART_RX: track 154.3 -> 0.00 mm, vias 4 -> 0
- net N: track 141.5 -> 0.00 mm
- net /N: track 0.00 -> 129.6 mm
- net /RS485_UART_RX: track 0.00 -> 122.3 mm, vias 0 -> 2
- net /ESP_U0RX: track 0.00 -> 121.2 mm, vias 0 -> 9
- net /RS485_UART_TX: track 0.00 -> 115.1 mm
- net /ESP_U0TX: track 0.00 -> 106.7 mm, vias 0 -> 7
- net /USB_VBUS: track 0.00 -> 87.0 mm, vias 0 -> 2
- net PE: track 81.9 -> 0.00 mm
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Other:
- board text removed: "D60-D63 STATUS"
- board text removed: "DNP IN TEMP VARIANT"

Commit message: sicherung
Parts:
- removed U6: CP2102N-A02-GQFN24, Package_DFN_QFN:QFN-24-1EP_4x4mm_P0.5mm_EP2.6x2.6mm
- added H1: MountingHole_M3, MountingHole:MountingHole_3.2mm_M3, F.Cu at (44.5, 37.0)
- added H2: MountingHole_M3, MountingHole:MountingHole_3.2mm_M3, F.Cu at (195.5, 36.2)
- added H3: MountingHole_M3, MountingHole:MountingHole_3.2mm_M3, F.Cu at (45.9, 136.6)
- added H4: MountingHole_M3, MountingHole:MountingHole_3.2mm_M3, F.Cu at (194.5, 137.9)
- added J5: EXT_GPIO_HEADER, PinHeader_2x10_P2.54mm_Vertical, F.Cu at (133.9, 36.7)
- added R90: 10k 1% 0603, Resistor_SMD:R_0603_1608Metric, F.Cu at (127.0, 43.5)
- added SW1: BOOT/CFG RESET, Button_Switch_SMD:SW_Push_1TS009xxxx-xxxx-xxxx_6x6x5mm, F.Cu at (137.1, 76.3)
- J3, J4: value 3-pin 3.5mm terminal -> KF128L-3.5-3P; footprint FW_Pumpengruppe:TB_3_350 -> FW_Pumpengruppe:TB_KF128L_350_3P
- K1: value G5LE-1A-E DC5 -> SRD-05VDC-SL-C; footprint FW_Pumpengruppe:Relay_SPST_16A -> Relay_SPDT_SANYOU_SRD_Series_Form_C
- K2: value G5LE-1A-E DC5 -> SRD-05VDC-SL-C; footprint FW_Pumpengruppe:Relay_SPST_8A -> Relay_SPDT_SANYOU_SRD_Series_Form_C
- K3: value G5LE-1 DC5 -> SRD-05VDC-SL-C; footprint FW_Pumpengruppe:Relay_SPDT_8A -> Relay_SPDT_SANYOU_SRD_Series_Form_C
- PSU1: value IRM-05-5 -> HLK-5M05; footprint Converter_ACDC:Converter_ACDC_MeanWell_IRM-05-xx_THT -> Converter_ACDC:Converter_ACDC_Hi-Link_HLK-5Mxx
- U1: value ESP32-WROOM-32D-N4 -> ESP32-S3-WROOM-1-N4; footprint RF_Module:ESP32-WROOM-32D -> ESP32-S3-WROOM-1
- X1, X2: value 3-pin 7.62mm terminal -> KF128-5.08-3P-AA; footprint FW_Pumpengruppe:TB_3_762 -> FW_Pumpengruppe:TB_KF128_508_3P
- X3: value 4-pin 7.62mm terminal -> DB128L-5.08-4P-GN-S; footprint FW_Pumpengruppe:TB_4_762 -> FW_Pumpengruppe:TB_DB128L_508_4P
- X4, X5: value 2-pin 3.5mm terminal -> KF128L-3.5-2P; footprint FW_Pumpengruppe:TB_2_350 -> FW_Pumpengruppe:TB_KF128L_350_2P
- moved RV1 50.6 mm to (45.2, 65.2)
- moved U5 34.5 mm to (103.0, 42.0)
- moved F1 27.8 mm to (59.1, 50.1)
- moved R60 18.8 mm to (152.9, 58.4)
- moved C23 12.9 mm to (187.4, 48.0), turned to 0 degrees
- moved X3 7.86 mm to (44.7, 116.5)
- moved D3 7.48 mm to (99.4, 125.0)
- moved K1 7.00 mm to (88.0, 83.0), turned to 180 degrees
- moved K2 7.00 mm to (88.0, 105.0), turned to 180 degrees
- moved K3 7.00 mm to (88.0, 125.0), turned to 180 degrees
- moved X2 6.93 mm to (44.6, 92.1)
- moved D2 5.85 mm to (100.0, 104.0)
- moved Q1 5.73 mm to (105.1, 81.5)
- moved R33 5.61 mm to (142.9, 36.5), turned to 0 degrees
- moved U1 5.42 mm to (154.7, 39.2)
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Connections:
- D83 pad 1: unconnected-(D83-DOUT-Pad1) -> (no net)
- J1 pad 3: unconnected-(J1-Pin_3-Pad3) -> (no net)
- J1 pad 6: unconnected-(J1-Pin_6-Pad6) -> (no net)
- J2 pad 3: unconnected-(J2-Pin_3-Pad3) -> (no net)
- J2 pad 6: unconnected-(J2-Pin_6-Pad6) -> (no net)
- JP1 pad 3: unconnected-(JP1-Pin_3-Pad3) -> (no net)
- K1 pad 2: /L_PUMP -> /+5V
- K2 pad 2: /L_MIX_ENABLE -> /+5V
- R33 pad 1: /ESP_EN -> /+3V3
- R33 pad 2: /+3V3 -> /ESP_EN
- U1 pad 10: /PUMP_DRV_GPIO -> /RS485_UART_TX
- U1 pad 11: /MIX_ENABLE_DRV_GPIO -> /ESP_IO18_EXT
- U1 pad 12: /MIX_DIR_DRV_GPIO -> /ESP_IO8_EXT
- U1 pad 13: unconnected-(U1-IO14-Pad13) -> /USB_D-
- U1 pad 14: unconnected-(U1-IO12-Pad14) -> /USB_D+
- U1 pad 15: /GND -> /ESP_IO3_EXT
- U1 pad 16: unconnected-(U1-IO13-Pad16) -> /ESP_IO46_EXT
- U1 pad 17: unconnected-(U1-SHD/SD2-Pad17) -> /RTD_RL_CS
- U1 pad 18: unconnected-(U1-SWP/SD3-Pad18) -> /RTD_VL_CS
- U1 pad 19: unconnected-(U1-SCS/CMD-Pad19) -> /SPI_MOSI
- U1 pad 20: unconnected-(U1-SCK/CLK-Pad20) -> /SPI_SCK
- U1 pad 21: unconnected-(U1-SDO/SD0-Pad21) -> /SPI_MISO
- U1 pad 22: unconnected-(U1-SDI/SD1-Pad22) -> /ESP_IO14_EXT
- U1 pad 23: unconnected-(U1-IO15-Pad23) -> /RGB_DATA
- U1 pad 24: unconnected-(U1-IO2-Pad24) -> /ESP_IO47_EXT
- U1 pad 25: unconnected-(U1-IO0-Pad25) -> /ESP_IO48_EXT
- U1 pad 26: /RS485_DE -> /ESP_IO45_EXT
- U1 pad 27: /RS485_UART_RX -> /ESP_IO0_BOOT
- U1 pad 28: /RS485_UART_TX -> /PUMP_DRV_GPIO
- U1 pad 29: /RTD_VL_CS -> /MIX_ENABLE_DRV_GPIO
- U1 pad 30: /SPI_SCK -> /MIX_DIR_DRV_GPIO
- U1 pad 31: /SPI_MISO -> /ESP_IO38_EXT
- U1 pad 32: unconnected-(U1-NC-Pad32) -> /ESP_IO39_EXT
- U1 pad 33: /RGB_DATA -> /ESP_IO40_EXT
- U1 pad 34: /ESP_U0RX -> /ESP_IO41_EXT
- U1 pad 35: /ESP_U0TX -> /ESP_IO42_EXT
- U1 pad 36: /RTD_RL_CS -> /ESP_RXD0_EXT
- U1 pad 37: /SPI_MOSI -> /ESP_TXD0_EXT
- U1 pad 38: /GND -> /ESP_IO2_EXT
- U1 pad 39: /GND -> /ESP_IO1_EXT
- U1 pad 4: unconnected-(U1-SENSOR_VP-Pad4) -> /RS485_DE
- U1 pad 5: unconnected-(U1-SENSOR_VN-Pad5) -> /ESP_IO5_EXT
- U1 pad 6: unconnected-(U1-IO34-Pad6) -> /ESP_IO6_EXT
- U1 pad 7: unconnected-(U1-IO35-Pad7) -> /ESP_IO7_EXT
- U1 pad 8: unconnected-(U1-IO32-Pad8) -> /ESP_IO15_EXT
- U1 pad 9: unconnected-(U1-IO33-Pad9) -> /RS485_UART_RX
- U2 pad 1: unconnected-(U2-~{DRDY}-Pad1) -> (no net)
- U2 pad 20: unconnected-(U2-NC-Pad20) -> (no net)
- U3 pad 1: unconnected-(U3-~{DRDY}-Pad1) -> (no net)
- U3 pad 20: unconnected-(U3-NC-Pad20) -> (no net)
- X6 pad A8: unconnected-(X6-SBU1-PadA8) -> (no net)
- X6 pad B8: unconnected-(X6-SBU2-PadB8) -> (no net)
Routing:
- net /PUMP_DRV_GPIO: track 83.1 -> 228.8 mm
- net /USB_D-: track 16.1 -> 151.2 mm, vias 2 -> 4
- net /USB_D+: track 15.6 -> 148.7 mm, vias 2 -> 4
- net /ESP_U0RX: track 121.2 -> 0.00 mm, vias 9 -> 0
- net /ESP_IO0_BOOT: track 0.00 -> 117.4 mm, vias 0 -> 4
- net /MIX_ENABLE_DRV_GPIO: track 104.1 -> 211.2 mm
- net /ESP_U0TX: track 106.7 -> 0.00 mm, vias 7 -> 0
- net /MIX_DIR_DRV_GPIO: track 121.8 -> 197.3 mm
- net /GND: track 720.0 -> 659.0 mm, vias 8 -> 15
- net /ESP_IO42_EXT: track 0.00 -> 57.2 mm, vias 0 -> 3
- net /+5V: track 529.5 -> 583.9 mm, vias 6 -> 1
- net /ESP_IO41_EXT: track 0.00 -> 52.6 mm, vias 0 -> 3
- net /ESP_IO40_EXT: track 0.00 -> 52.5 mm, vias 0 -> 1
- net /ESP_IO39_EXT: track 0.00 -> 44.7 mm, vias 0 -> 3
- net /ESP_IO38_EXT: track 0.00 -> 44.7 mm, vias 0 -> 1
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Other:
- outline, holes or cut-outs redrawn
- board text removed: "8mm+ ISOLATION SLOT / KEEP OUT"

Commit message: sicherung
Parts:
- F1: value 5x20 fuse holder -> 2x FC-203-22 fuse clips for 5x20
- U4: value MAX3485EESA+ -> SP3485EN-L/TR
Changed lines of the file:
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@@
 			)
 		)
-		(property "Supplier" "AISLER source or equivalent"
+		(property "Supplier" "LCSC C8963 / PCBWay equivalent"
 			(at 0 0 0)
 			(unlocked yes)
@@
 			)
 		)
-		(property "Value" "MAX3485EESA+"
+		(property "Value" "SP3485EN-L/TR"
 			(at 0 3.4 0)
 			(layer "F.Fab")
@@
 			)
 		)
-		(property "Manufacturer" "Analog Devices"
+		(property "Manufacturer" "MaxLinear"
 			(at 0 0 0)
 			(unlocked yes)
@@
 			)
 		)
-		(property "MPN" "MAX3485EESA+"
+		(property "MPN" "SP3485EN-L/TR"
 			(at 0 0 0)
 			(unlocked yes)
@@
 			)
 		)
-		(property "Supplier" "AISLER source or equivalent"
+		(property "Supplier" "LCSC C8963 / PCBWay equivalent"
 			(at 0 0 0)
 			(unlocked yes)
@@
 			)
 		)
-		(property "AISLER_MPN" "MAX3485EESA+"
+		(property "AISLER_MPN" "SP3485EN-L/TR"
 			(at 0 0 0)
 			(unlocked yes)
@@
 		(layer "F.Cu")
 		(at 127 43.5)
-		(descr "Resistor SMD 0603 boot pull-up")
+		(descr "Resistor SMD 0603 (1608 Metric), square (rectangular) end terminal, IPC-7351 nominal, (Body size source: IPC-SM-782 page 72, https://www.pcb-3d.com/wordpress/wp-content/uploads/ipc-sm-782a_amendment_1_and_2.pdf)")
+		(tags "resistor")
 		(property "Reference" "R90"
 			(at 0 -1.43 0)
@@
 			)
 		)
-		(property "Manufacturer" "Yageo"
+		(property "KiLib_Generator" "Yageo"
 			(at 0 0 0)
 			(layer "F.Fab")
@@
 		(duplicate_pad_numbers_are_jumpers no)
 		(fp_line
-			(start -0.14058 -0.51)
-			(end 0.14058 -0.51)
+			(start -0.237258 -0.5225)
+			(end 0.237258 -0.5225)
 			(stroke
 				(width 0.12)
@@
 		)
 		(fp_line
-			(start -0.14058 0.51)
-			(end 0.14058 0.51)
+			(start -0.237258 0.5225)
+			(end 0.237258 0.5225)
 			(stroke
 				(width 0.12)
@@
 		)
 		(fp_rect
-			(start -0.8 -0.4)
-			(end 0.8 0.4)
+			(start -0.8 -0.4125)
+			(end 0.8 0.4125)
 			(stroke
 				(width 0.1)
@@
 		)
 		(pad "1" smd roundrect
-			(at -0.775 0)
-			(size 0.9 0.95)
+			(at -0.825 0)
+			(size 0.8 0.95)
 			(layers "F.Cu" "F.Mask" "F.Paste")
 			(roundrect_rratio 0.25)
@@
 		)
 		(pad "2" smd roundrect
-			(at 0.775 0)
-			(size 0.9 0.95)
+			(at 0.825 0)
+			(size 0.8 0.95)
 			(layers "F.Cu" "F.Mask" "F.Paste")
 			(roundrect_rratio 0.25)
@@
 		(layer "F.Cu")
 		(at 44.9 51.9)
-		(descr "Cixi Kefa KF128-5.08-3P-AA, side-entry top-screw terminal")
+		(descr "Cixi Kefa KF128-5.08-3P-AA, 3-pin 5.08 mm side-entry top-screw terminal")
+		(tags "screw terminal 5.08mm 3P side-entry top-screw")
 		(property "Reference" "X1"
 			(at -0.1 -9.8 0)
@@
 		(attr through_hole)
 		(duplicate_pad_numbers_are_jumpers no)
+		(fp_line
+			(start -7.2 -8.6)
+			(end -7.2 8.6)
+			(stroke
+				(width 0.12)
+				(type solid)
+			)
+			(layer "F.SilkS")
+		)
+		(fp_line
+			(start -4.8 -8.6)
+			(end -7.2 -8.6)
+			(stroke
+				(width 0.12)
+				(type solid)
+			)
+			(layer "F.SilkS")
+		)
+		(fp_line
+			(start -4.8 8.6)
+			(end -7.2 8.6)
+			(stroke
+				(width 0.12)
+				(type solid)
+			)
+			(layer "F.SilkS")
+		)
 		(fp_rect
 			(start -4.8 -8.6)
@@
 			)
 		)
-		(property "Value" "5x20 fuse holder"
+		(property "Value" "2x FC-203-22 fuse clips for 5x20"
 			(at 8.9 7 270)
 			(layer "F.Fab")
@@
 			)
 		)
-		(property "Manufacturer" "Littelfuse"
+		(property "Manufacturer" "Bel Fuse"
 			(at 0 3.5 0)
 			(layer "F.Fab")
@@
 			)
 		)
-		(property "MPN" "03453LS1H"
+		(property "MPN" "FC-203-22"
 			(at 0 5 0)
 			(layer "F.Fab")
@@
 			)
 		)
-		(property "AISLER_MPN" "03453LS1H"
+		(property "AISLER_MPN" "FC-203-22"
 			(at 0 6.5 0)
 			(layer "F.Fab")
@@
 			)
 		)
-		(property "Supplier" "AISLER source or equivalent"
+		(property "Supplier" "LCSC C3205463 / PCBWay equivalent"
 			(at 0 0 270)
 			(unlocked yes)
@@
 			)
 		)
-		(property "AssemblyNote" "5x20 PCB fuse holder/fuse solution, verify footprint and fuse rating before order"
+		(property "AssemblyNote" "Populate two FC-203-22 clips per F1 footprint for one 5x20mm fuse; do not use one-piece expensive fuse holder"
 			(at 0 0 270)
 			(unlocked yes)
@@
 		(layer "F.Cu")
 		(at 44.6 92.08)
-		(descr "Cixi Kefa KF128-5.08-3P-AA, side-entry top-screw terminal")
+		(descr "Cixi Kefa KF128-5.08-3P-AA, 3-pin 5.08 mm side-entry top-screw terminal")
+		(tags "screw terminal 5.08mm 3P side-entry top-screw")
 		(property "Reference" "X2"
 			(at 0 -9.88 0)
@@
 		(attr through_hole)
 		(duplicate_pad_numbers_are_jumpers no)
+		(fp_line
+			(start -7.2 -8.6)
+			(end -7.2 8.6)
+			(stroke
+				(width 0.12)
+				(type solid)
+			)
+			(layer "F.SilkS")
+		)
+		(fp_line
+			(start -4.8 -8.6)
+			(end -7.2 -8.6)
+			(stroke
+				(width 0.12)
+				(type solid)
+			)
+			(layer "F.SilkS")
+		)
+		(fp_line
+			(start -4.8 8.6)
+			(end -7.2 8.6)
+			(stroke
+				(width 0.12)
+				(type solid)
+			)
+			(layer "F.SilkS")
+		)
 		(fp_rect
 			(start -4.8 -8.6)
@@
 		(layer "F.Cu")
 		(at 44.7 116.52)
-		(descr "DORABO DB128L-5.08-4P-GN-S, side-entry top-screw terminal")
+		(descr "DORABO DB128L-5.08-4P-GN-S, 4-pin 5.08 mm side-entry top-screw terminal")
+		(tags "screw terminal 5.08mm 4P side-entry top-screw")
 		(property "Reference" "X3"
 			(at 0.1 -12.32 0)
@@
 		(attr through_hole)
 		(duplicate_pad_numbers_are_jumpers no)
+		(fp_line
+			(start -7.2 -11.2)
+			(end -7.2 11.2)
+			(stroke
+				(width 0.12)
+				(type solid)
+			)
+			(layer "F.SilkS")
+		)
+		(fp_line
+			(start -4.8 -11.2)
+			(end -7.2 -11.2)
+			(stroke
+				(width 0.12)
+				(type solid)
+			)
+			(layer "F.SilkS")
+		)
+		(fp_line
+			(start -4.8 11.2)
+			(end -7.2 11.2)
+			(stroke
+				(width 0.12)
+				(type solid)
+			)
+			(layer "F.SilkS")
+		)
 		(fp_rect
 			(start -4.8 -11.2)
@@
 		(tags "SOT TO_SOT_SMD")
 		(property "Reference" "Q2"
-			(at 0.5 -5.4 0)
+			(at 0.1875 -2.45 0)
 			(layer "F.SilkS")
 			(effects
@@
 		(layer "F.Cu")
 		(at 142.9 36.5)
-		(descr "Resistor SMD 0603 (1608 Metric), square (rectangular) end terminal, IPC-7351 nominal")
+		(descr "Resistor SMD 0603 (1608 Metric), square (rectangular) end terminal, IPC-7351 nominal, (Body size source: IPC-SM-782 page 72, https://www.pcb-3d.com/wordpress/wp-content/uploads/ipc-sm-782a_amendment_1_and_2.pdf)")
 		(tags "resistor")
 		(property "Reference" "R33"
@@
 			)
 		)
-		(property "Manufacturer" "Yageo"
-			(at 0 3.5 180)
+		(property "KiLib_Generator" "AISLER source or equivalent"
+			(at 0 0 180)
+			(unlocked yes)
 			(layer "F.Fab")
 			(hide yes)
@@
 			)
 		)
-		(property "MPN" "RC0603FR-0710KL"
-			(at 0 5 180)
+		(property "Manufacturer" "Yageo"
+			(at 0 3.5 180)
 			(layer "F.Fab")
 			(hide yes)
@@
 			)
 		)
-		(property "AISLER_MPN" "RC0603FR-0710KL"
-			(at 0 6.5 180)
+		(property "MPN" "RC0603FR-0710KL"
+			(at 0 5 180)
 			(layer "F.Fab")
 			(hide yes)
@@
 			)
 		)
-		(property "Supplier" "AISLER source or equivalent"
-			(at 0 0 180)
-			(unlocked yes)
+		(property "AISLER_MPN" "RC0603FR-0710KL"
+			(at 0 6.5 180)
 			(layer "F.Fab")
 			(hide yes)
@@
 		)
 		(pad "1" smd roundrect
-			(at -0.825 0 180)
+			(at -0.825 0)
 			(size 0.8 0.95)
 			(layers "F.Cu" "F.Mask" "F.Paste")
@@
 		)
 		(pad "2" smd roundrect
-			(at 0.825 0 180)
+			(at 0.825 0)
 			(size 0.8 0.95)
 			(layers "F.Cu" "F.Mask" "F.Paste")
@@
 		(layer "Edge.Cuts")
 	)
-	(gr_text "RJ45: 1/2=5V 3/6=NC 4=A 5=B 7/8=GND"
-		(at 165 140 0)
+	(gr_text "GND"
+		(at 188.5 61 0)
 		(layer "F.SilkS")
 		(effects
@@
 	)
 	(gr_text "GND"
-		(at 188.5 61 0)
+		(at 189 108.5 0)
 		(layer "F.SilkS")
 		(effects
@@
 		)
 	)
-	(gr_text "GND"
-		(at 189 108.5 0)
+	(gr_text "RJ45: 1/2=5V 3/6=NC 4=A 5=B 7/8=GND"
+		(at 165 140 0)
 		(layer "F.SilkS")
 		(effects
 			(font
 				(size 0.65 0.65)
-				(thickness 0.1)
+				(thickness 0.254)
 			)
 		)
