File: hardware/pumpengruppe-rs485/pumpengruppe-rs485.kicad_sch (KiCad schematic)
At the start: 23 parts, among them J1 RJ45_RS485_IN, J2 RJ45_RS485_OUT, J3 YSTY_RS485_IN, J4 YSTY_RS485_OUT, K1 RELAY_PUMPE_16A, K2 RELAY_MISCHER_AUF, K3 RELAY_MISCHER_ZU, U1 ESP32-WROOM-32U, U2 MAX31865_VL, U3 MAX31865_RL, U4 ISOLATED_RS485, U6 CP2102N_USB_UART, X1 230V_IN_L_N_PE, X2 PUMPE_L_SW_N_PE, X3 MISCHER_AUF_ZU_N_PE, X4 RTD_VL_PT1000, X5 RTD_RL_PT1000, X6 USB_C_SERVICE_FLASH

Commit message: sicherung
Parts:
- added F1: TBD_T2A_T4A_L_FUSED, FW_Pumpengruppe:FUSE_5X20, symbol FW_Pumpengruppe:FUSE_2
- added U5: 3V3_REG, FW_Pumpengruppe:LDO_SOT223, symbol FW_Pumpengruppe:LDO_3V3
- K1, K2, K3: symbol FW_Pumpengruppe:BLOCK_4 -> FW_Pumpengruppe:RELAY_SPST_COIL
- PSU1: symbol FW_Pumpengruppe:BLOCK_4 -> FW_Pumpengruppe:ACDC_230_5V
- U1: symbol FW_Pumpengruppe:BLOCK_8 -> FW_Pumpengruppe:ESP32_PUMPCTRL
- U2, U3: symbol FW_Pumpengruppe:BLOCK_4 -> FW_Pumpengruppe:MAX31865_MIN
- U4: symbol FW_Pumpengruppe:BLOCK_4 -> FW_Pumpengruppe:ISO_RS485_6
- U6: symbol FW_Pumpengruppe:BLOCK_4 -> FW_Pumpengruppe:USB_UART_MIN
- X6: symbol FW_Pumpengruppe:CONN_4 -> FW_Pumpengruppe:USB_C_SERVICE_MIN
Changed lines of the file:
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@@
     (property "Footprint" "FW_Pumpengruppe:TB_3_762" (at 35 67 0) (effects (font (size 1.27 1.27)) hide))
+  )
+  (symbol (lib_id "FW_Pumpengruppe:FUSE_2") (at 55 55 0) (unit 1)
+    (exclude_from_sim no) (in_bom yes) (on_board yes) (dnp no)
+    (property "Reference" "F1" (at 55 49 0) (effects (font (size 1.27 1.27))))
+    (property "Value" "TBD_T2A_T4A_L_FUSED" (at 55 61 0) (effects (font (size 1.27 1.27))))
+    (property "Footprint" "FW_Pumpengruppe:FUSE_5X20" (at 55 65 0) (effects (font (size 1.27 1.27)) hide))
   )
   (symbol (lib_id "FW_Pumpengruppe:CONN_3") (at 35 90 0) (unit 1)
@@
     (property "Footprint" "FW_Pumpengruppe:TB_4_762" (at 35 138 0) (effects (font (size 1.27 1.27)) hide))
   )
-  (symbol (lib_id "FW_Pumpengruppe:BLOCK_4") (at 70 55 0) (unit 1)
+  (symbol (lib_id "FW_Pumpengruppe:ACDC_230_5V") (at 80 55 0) (unit 1)
     (exclude_from_sim no) (in_bom yes) (on_board yes) (dnp no)
-    (property "Reference" "PSU1" (at 70 44 0) (effects (font (size 1.27 1.27))))
-    (property "Value" "ACDC_230VAC_5V_ISOLATED" (at 70 66 0) (effects (font (size 1.27 1.27))))
-    (property "Footprint" "FW_Pumpengruppe:ACDC_IRM05" (at 70 70 0) (effects (font (size 1.27 1.27)) hide))
+    (property "Reference" "PSU1" (at 80 44 0) (effects (font (size 1.27 1.27))))
+    (property "Value" "ACDC_230VAC_5V_ISOLATED" (at 80 66 0) (effects (font (size 1.27 1.27))))
+    (property "Footprint" "FW_Pumpengruppe:ACDC_IRM05" (at 80 70 0) (effects (font (size 1.27 1.27)) hide))
   )
-  (symbol (lib_id "FW_Pumpengruppe:BLOCK_4") (at 70 90 0) (unit 1)
+  (symbol (lib_id "FW_Pumpengruppe:RELAY_SPST_COIL") (at 70 90 0) (unit 1)
     (exclude_from_sim no) (in_bom yes) (on_board yes) (dnp no)
     (property "Reference" "K1" (at 70 79 0) (effects (font (size 1.27 1.27))))
@@
     (property "Footprint" "FW_Pumpengruppe:Relay_SPST_16A" (at 70 105 0) (effects (font (size 1.27 1.27)) hide))
   )
-  (symbol (lib_id "FW_Pumpengruppe:BLOCK_4") (at 70 120 0) (unit 1)
+  (symbol (lib_id "FW_Pumpengruppe:RELAY_SPST_COIL") (at 70 120 0) (unit 1)
     (exclude_from_sim no) (in_bom yes) (on_board yes) (dnp no)
     (property "Reference" "K2" (at 70 109 0) (effects (font (size 1.27 1.27))))
@@
     (property "Footprint" "FW_Pumpengruppe:Relay_SPST_8A" (at 70 135 0) (effects (font (size 1.27 1.27)) hide))
   )
-  (symbol (lib_id "FW_Pumpengruppe:BLOCK_4") (at 70 150 0) (unit 1)
+  (symbol (lib_id "FW_Pumpengruppe:RELAY_SPST_COIL") (at 70 150 0) (unit 1)
     (exclude_from_sim no) (in_bom yes) (on_board yes) (dnp no)
     (property "Reference" "K3" (at 70 139 0) (effects (font (size 1.27 1.27))))
@@
     (property "Footprint" "FW_Pumpengruppe:Relay_SPST_8A" (at 70 165 0) (effects (font (size 1.27 1.27)) hide))
   )
-  (symbol (lib_id "FW_Pumpengruppe:BLOCK_8") (at 140 75 0) (unit 1)
+  (symbol (lib_id "FW_Pumpengruppe:LDO_3V3") (at 110 55 0) (unit 1)
+    (exclude_from_sim no) (in_bom yes) (on_board yes) (dnp no)
+    (property "Reference" "U5" (at 110 47 0) (effects (font (size 1.27 1.27))))
+    (property "Value" "3V3_REG" (at 110 63 0) (effects (font (size 1.27 1.27))))
+    (property "Footprint" "FW_Pumpengruppe:LDO_SOT223" (at 110 67 0) (effects (font (size 1.27 1.27)) hide))
+  )
+  (symbol (lib_id "FW_Pumpengruppe:ESP32_PUMPCTRL") (at 140 75 0) (unit 1)
     (exclude_from_sim no) (in_bom yes) (on_board yes) (dnp no)
     (property "Reference" "U1" (at 140 59 0) (effects (font (size 1.27 1.27))))
@@
     (property "Footprint" "FW_Pumpengruppe:ESP32_WROOM_KEEP_OUT" (at 140 95 0) (effects (font (size 1.27 1.27)) hide))
   )
-  (symbol (lib_id "FW_Pumpengruppe:BLOCK_4") (at 110 120 0) (unit 1)
+  (symbol (lib_id "FW_Pumpengruppe:MAX31865_MIN") (at 110 120 0) (unit 1)
     (exclude_from_sim no) (in_bom yes) (on_board yes) (dnp no)
     (property "Reference" "U2" (at 110 109 0) (effects (font (size 1.27 1.27))))
@@
     (property "Footprint" "FW_Pumpengruppe:SOIC16_RTD" (at 110 135 0) (effects (font (size 1.27 1.27)) hide))
   )
-  (symbol (lib_id "FW_Pumpengruppe:BLOCK_4") (at 110 150 0) (unit 1)
+  (symbol (lib_id "FW_Pumpengruppe:MAX31865_MIN") (at 110 150 0) (unit 1)
     (exclude_from_sim no) (in_bom yes) (on_board yes) (dnp no)
     (property "Reference" "U3" (at 110 139 0) (effects (font (size 1.27 1.27))))
@@
     (property "Footprint" "FW_Pumpengruppe:SOIC16_RTD" (at 110 165 0) (effects (font (size 1.27 1.27)) hide))
   )
-  (symbol (lib_id "FW_Pumpengruppe:BLOCK_4") (at 180 75 0) (unit 1)
+  (symbol (lib_id "FW_Pumpengruppe:ISO_RS485_6") (at 180 75 0) (unit 1)
     (exclude_from_sim no) (in_bom yes) (on_board yes) (dnp no)
     (property "Reference" "U4" (at 180 64 0) (effects (font (size 1.27 1.27))))
@@
     (property "Footprint" "FW_Pumpengruppe:TB_2_350" (at 150 160 0) (effects (font (size 1.27 1.27)) hide))
   )
-  (symbol (lib_id "FW_Pumpengruppe:CONN_4") (at 185 42 0) (unit 1)
+  (symbol (lib_id "FW_Pumpengruppe:USB_C_SERVICE_MIN") (at 185 42 0) (unit 1)
     (exclude_from_sim no) (in_bom yes) (on_board yes) (dnp no)
     (property "Reference" "X6" (at 185 33 0) (effects (font (size 1.27 1.27))))
@@
     (property "Footprint" "FW_Pumpengruppe:USB_C_SERVICE" (at 185 55 0) (effects (font (size 1.27 1.27)) hide))
   )
-  (symbol (lib_id "FW_Pumpengruppe:BLOCK_4") (at 185 68 0) (unit 1)
+  (symbol (lib_id "FW_Pumpengruppe:USB_UART_MIN") (at 185 68 0) (unit 1)
     (exclude_from_sim no) (in_bom yes) (on_board yes) (dnp no)
     (property "Reference" "U6" (at 185 57 0) (effects (font (size 1.27 1.27))))
@@
   (symbol_instances
     (path "/877a40bb-a712-4421-9d1d-52c408dd5880" (reference "X1") (unit 1) (value "230V_IN_L_N_PE") (footprint "FW_Pumpengruppe:TB_3_762"))
+    (path "/a40ef0c2-343b-4610-b261-4cd71463784d" (reference "F1") (unit 1) (value "TBD_T2A_T4A_L_FUSED") (footprint "FW_Pumpengruppe:FUSE_5X20"))
     (path "/b6d9c439-385e-45f3-b924-96c1e1f6926c" (reference "X2") (unit 1) (value "PUMPE_L_SW_N_PE") (footprint "FW_Pumpengruppe:TB_3_762"))
     (path "/d155b36d-0c07-46df-ab01-10252b00b7a8" (reference "X3") (unit 1) (value "MISCHER_AUF_ZU_N_PE") (footprint "FW_Pumpengruppe:TB_4_762"))
@@
     (path "/978f8d56-c741-4af7-b591-94da6ed82b9c" (reference "K3") (unit 1) (value "RELAY_MISCHER_ZU") (footprint "FW_Pumpengruppe:Relay_SPST_8A"))
     (path "/dfae6d54-53f0-44f1-a454-c21c7c919d0c" (reference "U1") (unit 1) (value "ESP32-WROOM-32U") (footprint "FW_Pumpengruppe:ESP32_WROOM_KEEP_OUT"))
+    (path "/f14d5680-f3d7-458e-8017-db494be8a5a0" (reference "U5") (unit 1) (value "3V3_REG") (footprint "FW_Pumpengruppe:LDO_SOT223"))
     (path "/56f790cd-5f7f-4382-a8f3-f3c9bc06df1f" (reference "U2") (unit 1) (value "MAX31865_VL") (footprint "FW_Pumpengruppe:SOIC16_RTD"))
     (path "/9c525a1e-bd03-4ce1-b57d-d8962650e5ea" (reference "U3") (unit 1) (value "MAX31865_RL") (footprint "FW_Pumpengruppe:SOIC16_RTD"))

Commit message: sicherung
Parts:
- added C60, C61, C62, C63, C64, C65, C66, C67, C68, C69, C70, C71, C72, C73, C74, C75, C76, C77, C78, C79, C80, C81, C82, C83: 100n_RGB_LED, Capacitor_SMD:C_0603_1608Metric, symbol Device:C
- added D1: SS14_FLYBACK_PUMP, FW_Pumpengruppe:D_SOD123, symbol Device:D
- added D10: LED_PUMP, FW_Pumpengruppe:LED_0603, symbol Device:LED
- added D11: LED_MIX_ENABLE, FW_Pumpengruppe:LED_0603, symbol Device:LED
- added D12: LED_MIX_DIR, FW_Pumpengruppe:LED_0603, symbol Device:LED
- added D2: SS14_FLYBACK_MIX_ENABLE, FW_Pumpengruppe:D_SOD123, symbol Device:D
- added D20: LED_5V, FW_Pumpengruppe:LED_0603, symbol Device:LED
- added D21: LED_3V3, FW_Pumpengruppe:LED_0603, symbol Device:LED
- added D3: SS14_FLYBACK_MIX_DIR, FW_Pumpengruppe:D_SOD123, symbol Device:D
- added D30: LED_RS485_TX, FW_Pumpengruppe:LED_0603, symbol Device:LED
- added D31: LED_RS485_RX, FW_Pumpengruppe:LED_0603, symbol Device:LED
- added D4: SS14_USB_TO_5V, FW_Pumpengruppe:D_SOD123, symbol Device:D
- added D40: LED_230VAC, LED_SMD:LED_0805_2012Metric, symbol Device:LED
- added D41: 1N4148_LED_PROTECT, Diode_SMD:D_SOD-123, symbol Device:D
- added D50: TVS_RS485_A_COM, Diode_SMD:D_SOD-123, symbol Device:D_TVS
- added D51: TVS_RS485_B_COM, Diode_SMD:D_SOD-123, symbol Device:D_TVS
- added D52: TVS_RS485_A_B, Diode_SMD:D_SOD-123, symbol Device:D_TVS
- added D60: SK6812MINI_STATUS_1, LED_SMD:LED_SK6812MINI_PLCC4_3.5x3.5mm_P1.75mm, symbol LED:SK6812MINI
- added D61: SK6812MINI_STATUS_2, LED_SMD:LED_SK6812MINI_PLCC4_3.5x3.5mm_P1.75mm, symbol LED:SK6812MINI
- added D62: SK6812MINI_STATUS_3, LED_SMD:LED_SK6812MINI_PLCC4_3.5x3.5mm_P1.75mm, symbol LED:SK6812MINI
- added D63: SK6812MINI_STATUS_4, LED_SMD:LED_SK6812MINI_PLCC4_3.5x3.5mm_P1.75mm, symbol LED:SK6812MINI
- added D64: SK6812MINI_VALVE_5PCT, LED_SMD:LED_SK6812MINI_PLCC4_3.5x3.5mm_P1.75mm, symbol LED:SK6812MINI
- added D65: SK6812MINI_VALVE_10PCT, LED_SMD:LED_SK6812MINI_PLCC4_3.5x3.5mm_P1.75mm, symbol LED:SK6812MINI
- added D66: SK6812MINI_VALVE_15PCT, LED_SMD:LED_SK6812MINI_PLCC4_3.5x3.5mm_P1.75mm, symbol LED:SK6812MINI
- added D67: SK6812MINI_VALVE_20PCT, LED_SMD:LED_SK6812MINI_PLCC4_3.5x3.5mm_P1.75mm, symbol LED:SK6812MINI
- added D68: SK6812MINI_VALVE_25PCT, LED_SMD:LED_SK6812MINI_PLCC4_3.5x3.5mm_P1.75mm, symbol LED:SK6812MINI
- added D69: SK6812MINI_VALVE_30PCT, LED_SMD:LED_SK6812MINI_PLCC4_3.5x3.5mm_P1.75mm, symbol LED:SK6812MINI
- added D70: SK6812MINI_VALVE_35PCT, LED_SMD:LED_SK6812MINI_PLCC4_3.5x3.5mm_P1.75mm, symbol LED:SK6812MINI
- added D71: SK6812MINI_VALVE_40PCT, LED_SMD:LED_SK6812MINI_PLCC4_3.5x3.5mm_P1.75mm, symbol LED:SK6812MINI
- added D72: SK6812MINI_VALVE_45PCT, LED_SMD:LED_SK6812MINI_PLCC4_3.5x3.5mm_P1.75mm, symbol LED:SK6812MINI
- added D73: SK6812MINI_VALVE_50PCT, LED_SMD:LED_SK6812MINI_PLCC4_3.5x3.5mm_P1.75mm, symbol LED:SK6812MINI
- added D74: SK6812MINI_VALVE_55PCT, LED_SMD:LED_SK6812MINI_PLCC4_3.5x3.5mm_P1.75mm, symbol LED:SK6812MINI
- added D75: SK6812MINI_VALVE_60PCT, LED_SMD:LED_SK6812MINI_PLCC4_3.5x3.5mm_P1.75mm, symbol LED:SK6812MINI
- added D76: SK6812MINI_VALVE_65PCT, LED_SMD:LED_SK6812MINI_PLCC4_3.5x3.5mm_P1.75mm, symbol LED:SK6812MINI
- added D77: SK6812MINI_VALVE_70PCT, LED_SMD:LED_SK6812MINI_PLCC4_3.5x3.5mm_P1.75mm, symbol LED:SK6812MINI
- added D78: SK6812MINI_VALVE_75PCT, LED_SMD:LED_SK6812MINI_PLCC4_3.5x3.5mm_P1.75mm, symbol LED:SK6812MINI
- added D79: SK6812MINI_VALVE_80PCT, LED_SMD:LED_SK6812MINI_PLCC4_3.5x3.5mm_P1.75mm, symbol LED:SK6812MINI
- added D80: SK6812MINI_VALVE_85PCT, LED_SMD:LED_SK6812MINI_PLCC4_3.5x3.5mm_P1.75mm, symbol LED:SK6812MINI
- added D81: SK6812MINI_VALVE_90PCT, LED_SMD:LED_SK6812MINI_PLCC4_3.5x3.5mm_P1.75mm, symbol LED:SK6812MINI
- added D82: SK6812MINI_VALVE_95PCT, LED_SMD:LED_SK6812MINI_PLCC4_3.5x3.5mm_P1.75mm, symbol LED:SK6812MINI
- added D83: SK6812MINI_VALVE_100PCT, LED_SMD:LED_SK6812MINI_PLCC4_3.5x3.5mm_P1.75mm, symbol LED:SK6812MINI
- added F2: PTC_BUS_5V, Fuse:Fuse_1812_4532Metric, symbol Device:Polyfuse
- added Q1: AO3400A_PUMP, FW_Pumpengruppe:SOT23_NMOS, symbol Transistor_FET:Q_NMOS_GDS
- added Q2: AO3400A_MIX_ENABLE, FW_Pumpengruppe:SOT23_NMOS, symbol Transistor_FET:Q_NMOS_GDS
- added Q3: AO3400A_MIX_DIR, FW_Pumpengruppe:SOT23_NMOS, symbol Transistor_FET:Q_NMOS_GDS
- added R10: 2k2_LED_PUMP, FW_Pumpengruppe:R_0603, symbol Device:R
- added R11: 2k2_LED_MIX_ENABLE, FW_Pumpengruppe:R_0603, symbol Device:R
- added R12: 2k2_LED_MIX_DIR, FW_Pumpengruppe:R_0603, symbol Device:R
- added R20: 2k2_LED_5V, FW_Pumpengruppe:R_0603, symbol Device:R
- added R21: 1k5_LED_3V3, FW_Pumpengruppe:R_0603, symbol Device:R
- added R30: 4k7_LED_TX, FW_Pumpengruppe:R_0603, symbol Device:R
- added R31: 4k7_LED_RX, FW_Pumpengruppe:R_0603, symbol Device:R
- added R32: 0R_BUS_0V_LINK, FW_Pumpengruppe:R_0603, symbol Device:R
- added R4: 100R_GATE_PUMP, FW_Pumpengruppe:R_0603, symbol Device:R
- added R40: 150k_LED_230V_1, Resistor_SMD:R_1206_3216Metric, symbol Device:R
- added R41: 150k_LED_230V_2, Resistor_SMD:R_1206_3216Metric, symbol Device:R
- added R5: 100R_GATE_MIX_ENABLE, FW_Pumpengruppe:R_0603, symbol Device:R
- added R6: 100R_GATE_MIX_DIR, FW_Pumpengruppe:R_0603, symbol Device:R
- added R60: 330R_RGB_DATA, Resistor_SMD:R_0603_1608Metric, symbol Device:R
- added R7: 100k_GATE_PD_PUMP, FW_Pumpengruppe:R_0603, symbol Device:R
- added R8: 100k_GATE_PD_MIX_ENABLE, FW_Pumpengruppe:R_0603, symbol Device:R
- added R9: 100k_GATE_PD_MIX_DIR, FW_Pumpengruppe:R_0603, symbol Device:R
- added RV1: MOV_275VAC, Varistor:RV_Disc_D12mm_W3.9mm_P7.5mm, symbol Device:Varistor
- F1: symbol FW_Pumpengruppe:FUSE_2 -> Device:Fuse
- J1, J2: footprint FW_Pumpengruppe:RJ45_SHIELDED_GENERIC -> Connector_RJ:RJ45_Amphenol_54602-x08_Horizontal; symbol FW_Pumpengruppe:RJ45_8 -> Connector_Generic:Conn_01x08
- J3, J4, X1, X2: symbol FW_Pumpengruppe:CONN_3 -> Connector_Generic:Conn_01x03
- JP1: value RS485_TERM_ON -> RS485_TERM_ON_PARK; footprint FW_Pumpengruppe:JP_2_254 -> Connector_PinHeader_2.54mm:PinHeader_1x03_P2.54mm_Vertical; symbol FW_Pumpengruppe:CONN_2 -> Connector_Generic:Conn_01x03
- K2: value RELAY_MISCHER_AUF -> MIX_ENABLE_RELAY
- K3: value RELAY_MISCHER_ZU -> MIX_DIR_SPDT_RELAY; footprint FW_Pumpengruppe:Relay_SPST_8A -> FW_Pumpengruppe:Relay_SPDT_8A; symbol FW_Pumpengruppe:RELAY_SPST_COIL -> FW_Pumpengruppe:RELAY_SPDT_COIL
- PSU1: value ACDC_230VAC_5V_ISOLATED -> HLK-5M05; footprint FW_Pumpengruppe:ACDC_IRM05 -> Converter_ACDC:Converter_ACDC_Hi-Link_HLK-5Mxx; symbol FW_Pumpengruppe:ACDC_230_5V -> Converter_ACDC:HLK-5M05
- R1, R2, R3, X4, X5: symbol FW_Pumpengruppe:CONN_2 -> Connector_Generic:Conn_01x02
- U1: value ESP32-WROOM-32U -> ESP32-WROOM-32D; footprint FW_Pumpengruppe:ESP32_WROOM_KEEP_OUT -> RF_Module:ESP32-WROOM-32D; symbol FW_Pumpengruppe:ESP32_PUMPCTRL -> RF_Module:ESP32-WROOM-32
- U4: value ISOLATED_RS485 -> MAX3485; footprint FW_Pumpengruppe:ISO_RS485_MODULE -> Package_SO:SOIC-8_3.9x4.9mm_P1.27mm; symbol FW_Pumpengruppe:ISO_RS485_6 -> Interface_UART:MAX3485
- U5: symbol FW_Pumpengruppe:LDO_3V3 -> Regulator_Linear:AMS1117-3.3
- X3: symbol FW_Pumpengruppe:CONN_4 -> Connector_Generic:Conn_01x04
- X6: footprint FW_Pumpengruppe:USB_C_SERVICE -> Connector_USB:USB_C_Receptacle_HRO_TYPE-C-31-M-12; symbol FW_Pumpengruppe:USB_C_SERVICE_MIN -> Connector:USB_C_Receptacle_USB2.0_16P
Connections:
- new net: X6.A1 (GND), X6.A12 (GND), X6.B1 (GND), X6.B12 (GND)
- new net +3V3: R21.2, R30.2, R31.2, U1.1 (GND), U1.15 (GND), U1.38 (GND), U1.39 (GND), U2.9 (SCK), U3.9 (SCK)
- new net +5V: C60.1, C61.1, C62.1, C63.1, C64.1, C65.1, C66.1, C67.1, C68.1, C69.1, C70.1, C71.1, C72.1, C73.1, C74.1, C75.1, C76.1, C77.1, C78.1, C79.1, C80.1, C81.1, C82.1, C83.1, D1.1 (K), D2.1 (K), D3.1 (K), D4.1 (K), D60.4 (VDD), D61.4 (VDD), D62.4 (VDD), D63.4 (VDD), D64.4 (VDD), D65.4 (VDD), D66.4 (VDD), D67.4 (VDD), D68.4 (VDD), D69.4 (VDD), D70.4 (VDD), D71.4 (VDD), D72.4 (VDD), D73.4 (VDD), D74.4 (VDD), D75.4 (VDD), D76.4 (VDD), D77.4 (VDD), D78.4 (VDD), D79.4 (VDD), D80.4 (VDD), D81.4 (VDD), D82.4 (VDD), D83.4 (VDD), F2.1, K1.A2 (A2_DRV), K2.A2 (A2_DRV), K3.A2 (A2_DRV), R10.2, R11.2, R12.2, R20.2
- new net BUS_5V: F2.2, J1.6 (Pin_6), J1.7 (Pin_7), J2.6 (Pin_6), J2.7 (Pin_7)
- new net GND: C60.2, C61.2, C62.2, C63.2, C64.2, C65.2, C66.2, C67.2, C68.2, C69.2, C70.2, C71.2, C72.2, C73.2, C74.2, C75.2, C76.2, C77.2, C78.2, C79.2, C80.2, C81.2, C82.2, C83.2, D20.2 (A), D21.2 (A), D60.2 (VSS), D61.2 (VSS), D62.2 (VSS), D63.2 (VSS), D64.2 (VSS), D65.2 (VSS), D66.2 (VSS), D67.2 (VSS), D68.2 (VSS), D69.2 (VSS), D70.2 (VSS), D71.2 (VSS), D72.2 (VSS), D73.2 (VSS), D74.2 (VSS), D75.2 (VSS), D76.2 (VSS), D77.2 (VSS), D78.2 (VSS), D79.2 (VSS), D80.2 (VSS), D81.2 (VSS), D82.2 (VSS), D83.2 (VSS), Q1.3 (S), Q2.3 (S), Q3.3 (S), R32.1, R7.1, R8.1, R9.1, U1.2 (VDD), U2.1 (RTD+), U3.1 (RTD+), U6.1 (VBUS), X6.A4 (VBUS), X6.A9 (VBUS), X6.B4 (VBUS), X6.B9 (VBUS)
- new net LED230_A: D40.1 (K), D41.2 (A), R41.1
- new net LED230_DROP: R40.1, R41.2
- new net LED_3V3_A: D21.1 (K), R21.1
- new net LED_5V_A: D20.1 (K), R20.1
- new net LED_CLOSE_A: D12.1 (K), R12.1
- new net LED_OPEN_A: D11.1 (K), R11.1
- new net LED_PUMP_A: D10.1 (K), R10.1
- new net LED_RX_A: D31.1 (K), R31.1
- new net LED_TX_A: D30.1 (K), R30.1
- new net L_CLOSE: K3.NC (NC_ZU), X3.2 (Pin_2)
- new net L_FUSED: F1.1, K1.2 (NO), K2.2 (NO), R40.2, RV1.2
- new net L_IN: F1.2, X1.3 (Pin_3)
- new net L_OPEN: K3.C (COM), X3.3 (Pin_3)
- new net L_PUMP: K1.1 (COM), X2.3 (Pin_3)
- new net MIX_DIR_COIL_L: D12.2 (A), D3.2 (A), K3.A1 (A1_5V), Q3.2 (D)
- new net MIX_DIR_DRV: R6.2, U1.29 (IO5)
- new net MIX_DIR_GATE: Q3.1 (G), R6.1, R9.2
- new net MIX_ENABLE_COIL_L: D11.2 (A), D2.2 (A), K2.A1 (A1_5V), Q2.2 (D)
- new net MIX_ENABLE_DRV: R5.2, U1.14 (IO12)
- new net MIX_ENABLE_GATE: Q2.1 (G), R5.1, R8.2
- new net MIX_L_EN: K2.1 (COM), K3.NO (NO_AUF)
- new net N: D40.2 (A), D41.1 (K), RV1.1, X1.2 (Pin_2), X2.2 (Pin_2), X3.1 (Pin_1)
- new net PE: X1.1 (Pin_1), X2.1 (Pin_1)
- new net PUMP_COIL_L: D1.2 (A), D10.2 (A), K1.A1 (A1_5V), Q1.2 (D)
- new net PUMP_DRV: R4.2, U1.16 (IO13)
- new net PUMP_GATE: Q1.1 (G), R4.1, R7.2
- new net RGB_DATA: R60.1, U1.33 (IO21)
- new net RGB_DIN_1: D60.3 (DIN), R60.2
- new net RGB_DOUT_1: D60.1 (DOUT), D61.3 (DIN)
- new net RGB_DOUT_10: D69.1 (DOUT), D70.3 (DIN)
- new net RGB_DOUT_11: D70.1 (DOUT), D71.3 (DIN)
- new net RGB_DOUT_12: D71.1 (DOUT), D72.3 (DIN)
- new net RGB_DOUT_13: D72.1 (DOUT), D73.3 (DIN)
- new net RGB_DOUT_14: D73.1 (DOUT), D74.3 (DIN)
- new net RGB_DOUT_15: D74.1 (DOUT), D75.3 (DIN)
- new net RGB_DOUT_16: D75.1 (DOUT), D76.3 (DIN)
- new net RGB_DOUT_17: D76.1 (DOUT), D77.3 (DIN)
- new net RGB_DOUT_18: D77.1 (DOUT), D78.3 (DIN)
- new net RGB_DOUT_19: D78.1 (DOUT), D79.3 (DIN)
- new net RGB_DOUT_2: D61.1 (DOUT), D62.3 (DIN)
- new net RGB_DOUT_20: D79.1 (DOUT), D80.3 (DIN)
- new net RGB_DOUT_21: D80.1 (DOUT), D81.3 (DIN)
- new net RGB_DOUT_22: D81.1 (DOUT), D82.3 (DIN)
- new net RGB_DOUT_23: D82.1 (DOUT), D83.3 (DIN)
- new net RGB_DOUT_3: D62.1 (DOUT), D63.3 (DIN)
- new net RGB_DOUT_4: D63.1 (DOUT), D64.3 (DIN)
- new net RGB_DOUT_5: D64.1 (DOUT), D65.3 (DIN)
- new net RGB_DOUT_6: D65.1 (DOUT), D66.3 (DIN)
- new net RGB_DOUT_7: D66.1 (DOUT), D67.3 (DIN)
- new net RGB_DOUT_8: D67.1 (DOUT), D68.3 (DIN)
- new net RGB_DOUT_9: D68.1 (DOUT), D69.3 (DIN)
- new net RS485_A: D50.1 (A1), D52.1 (A1), J1.4 (Pin_4), J2.4 (Pin_4), J3.3 (Pin_3), J4.3 (Pin_3), R3.1 (Pin_1)
- new net RS485_B: D51.1 (A1), D52.2 (A2), J1.3 (Pin_3), J2.3 (Pin_3), J3.2 (Pin_2), J4.2 (Pin_2), JP1.2 (Pin_2)
- new net RS485_DE: U1.8 (IO32)
- new net RS485_GND: D50.2 (A2), D51.2 (A2), J1.1 (Pin_1), J2.1 (Pin_1), J3.1 (Pin_1), J4.1 (Pin_1), R32.2
- new net RS485_TERM: JP1.3 (Pin_3)
- new net RTD_RL_P: U3.8 (GND), X5.1 (Pin_1)
- new net RTD_VL_P: U2.8 (GND), X4.1 (Pin_1)
- new net SPI_MISO: U1.28 (IO17), U2.11 (MISO), U3.11 (MISO)
- new net SPI_MOSI: U1.13 (IO14)
- new net SPI_SCK: U1.30 (IO18), U2.16 (3V3), U3.16 (3V3)
- new net UART_RX: D31.2 (A), U1.9 (IO33), U6.7 (DTR_NC)
- new net UART_TX: D30.2 (A), U1.7 (IO35), U6.6 (RXD_FROM_ESP_TX)
- new net USB_CC1: R1.1 (Pin_1)
- new net USB_CC2: R2.1 (Pin_1)
- new net USB_D+: X6.A7 (D-)
- new net USB_D-: U6.3 (USB_D-), X6.A6 (D+), X6.B7 (D-)
- new net USB_VBUS: D4.2 (A), U6.4 (GND), X6.B8 (SBU2)
- no-connect marks 0 -> 26
Other:
- note added: "BUS / SERVICE U4 MAX3485/SP3485: A=RS485_A, B=RS485_B, COM ueber R32 zu lokal GND J1/J2 RJ45 parallel: Pin 4=D+, Pin 5=D-, Pin 1/2=BUS_5V, Pin 7/8=COM F2 PTC koppelt BUS_5V an lokal +5V; R32 koppelt COM an lokal GND fuer RJ45-5V-Versorgung X6 USB-C speist +5V ueber D4 Schottky J3/J4 YSTY parallel: D+, D-, COM R3 120R + JP1 1x3: 1-2 Abschluss EIN, 2-3 Park/AUS TX/RX, diskrete 230V-LED, 5V und 3V3 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"
- note added: "NETZ-/LASTLOGIK X1.1 L_IN -> F1 -> L_FUSED X1.2 N -> X2.2, X3.3, PSU1.N X1.3 PE -> X2.3, X3.4 K1: L_FUSED -> L_PUMP -> X2.1 K2 Mischer-Enable: L_FUSED -> MIX_L_EN K3 SPDT Richtung: MIX_L_EN -> NC=ZU / NO=AUF Damit sind AUF und ZU hardwareseitig gegeneinander verriegelt."
- note added: "RELAIS-TREIBER / ANZEIGEN / POWER-ORING Alle Relais: ESP GPIO -> 100R -> AO3400A Gate, 100k Pulldown, Spule nach +5V, SS14 Freilaufdiode. Status-LEDs liegen parallel zur jeweiligen Spulenansteuerung. TX/RX LEDs leuchten bei Low-Pulsen. K2/K3: K2 gibt Mischer-L frei; K3 ist SPDT Richtung NC=ZU / NO=AUF."
- note added: "SELV / CONTROL ZONE - U1: ESP32-WROOM-32D, PCB-Antenne am Platinenrand/Keepout - X6/U6: USB-C Service + USB-UART fuer Firmware/Debug - U2/U3: MAX31865 RTD VL/RL - U4: MAX3485/SP3485 RS485-Standardtransceiver, DE/RE per RS485_DE - J1/J2 RJ45 + J3/J4 Schraubklemmen liegen parallel - WLAN nur Konfiguration/OTA, Regelbetrieb ueber Modbus RTU"
- note added: "SELV-/MCU-LOGIK PSU1 HLK-5M05 5V -> U5 -> 3V3 U1 ESP32-WROOM-32D: PCB-Antenne am Platinenrand/Keepout U1 GPIO25/26/27 -> NMOS-Treiber: PUMP_DRV, MIX_ENABLE_DRV, MIX_DIR_DRV; GPIO4=RS485_DE Treiber je Relais: 100R Gate, 100k Pulldown, AO3400A, SS14 Freilauf, Status-LED U2/U3 MAX31865: VSPI GPIO23=MOSI, GPIO19=MISO, GPIO18=SCK X4 RTD_VL_P/N, X5 RTD_RL_P/N"
- note removed: "BUS / SERVICE U4 isolierter RS485: A=RS485_A, B=RS485_B, COM=RS485_GND J1/J2 RJ45 parallel: Pin 4=D+, Pin 5=D-, Pin 7/8=COM J3/J4 YSTY parallel: D+, D-, COM R3 120R + JP1: schaltbarer Abschluss zwischen A und B X6 USB-C -> U6 USB-UART -> U1 UART_TX/RX; CC1/CC2 je 5k1 nach GND"
- note removed: "NETZ-/LASTLOGIK X1.1 L_IN -> F1 -> L_FUSED X1.2 N -> X2.2, X3.3, PSU1.N X1.3 PE -> X2.3, X3.4 K1: L_FUSED -> L_PUMP -> X2.1 K2: L_FUSED -> L_OPEN -> X3.1 K3: L_FUSED -> L_CLOSE -> X3.2 K2/K3 zusaetzlich per Firmware und Treiber verriegeln."
- note removed: "SELV / CONTROL ZONE - U1: ESP32-WROOM-32U, Antenne extern ueber U.FL - X6/U6: USB-C Service + USB-UART fuer Firmware/Debug - U2/U3: MAX31865 RTD VL/RL - U4: isolierter RS485 - J1/J2 RJ45 + J3/J4 Schraubklemmen liegen parallel - WLAN nur Konfiguration/OTA, Regelbetrieb ueber Modbus RTU"
- note removed: "SELV-/MCU-LOGIK PSU1 5V -> U5 -> 3V3 U1 ESP32-WROOM-32U: externe Antenne per U.FL U1 GPIO -> Relaistreiber: PUMP_DRV, OPEN_DRV, CLOSE_DRV U2/U3 MAX31865: SPI_MOSI, SPI_MISO, SPI_SCK X4 RTD_VL_P/N, X5 RTD_RL_P/N"
