File: hardware/pumpengruppe-rs485/pumpengruppe-rs485.kicad_sch (KiCad schematic)
At the start: 111 parts, among them J1 RJ45 8P8C horizontal, J2 RJ45 8P8C horizontal, J3 3-pin 3.5mm terminal, J4 3-pin 3.5mm terminal, K1 G5LE-1A-E DC5, K2 G5LE-1A-E DC5, K3 G5LE-1 DC5, Q1 AO3400A, Q2 AO3400A, Q3 AO3400A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

Commit message: sicherung
Connections:
- net RGB_DATA: now also U1.27 (IO16); no longer U1.33 (IO21)
- net RS485_UART_TX: now reaches U1.31 (IO19)
- net RS485_UART_TX: now also D30.2 (A)
- net UART_RX renamed ESP_U0RX
- net ESP_U0RX: no longer D31.2 (A)
- net UART_TX renamed ESP_U0TX
- net ESP_U0TX: no longer D30.2 (A)
- new net RS485_UART_RX: D31.2 (A), U1.33 (IO21)
- no-connect marks 26 -> 25
