File: hardware/pumpengruppe-rs485/pumpengruppe-rs485.kicad_sch (KiCad schematic)
At the start: 111 parts, among them J1 RJ45 8P8C horizontal, J2 RJ45 8P8C horizontal, J3 3-pin 3.5mm terminal, J4 3-pin 3.5mm terminal, K1 G5LE-1A-E DC5, K2 G5LE-1A-E DC5, K3 G5LE-1 DC5, Q1 AO3400A, Q2 AO3400A, Q3 AO3400A, U1 ESP32-WROOM-32D-N4, U2 MAX31865AAP+, U3 MAX31865AAP+, U4 MAX3485EESA+, U5 AMS1117-3.3, U6 CP2102N-A02-GQFN24, X1 3-pin 7.62mm terminal, X2 3-pin 7.62mm terminal, X3 4-pin 7.62mm terminal, X4 2-pin 3.5mm terminal, X5 2-pin 3.5mm terminal, X6 USB-C receptacle

Commit message: sicherung
Parts:
- added C22, C23: 10nF 50V, Capacitor_SMD:C_0603_1608Metric, symbol Device:C
- added R22, R23: 4.3k 0.1% 0603, Resistor_SMD:R_0603_1608Metric, symbol Device:R
- added R33: 10k 1% 0603, Resistor_SMD:R_0603_1608Metric, symbol Device:R
- U2, U3: footprint Package_SO:SOIC-16_3.9x9.9mm_P1.27mm -> Package_SO:SSOP-20_5.3x7.2mm_P0.65mm; symbol FW_Pumpengruppe:MAX31865_MIN -> Sensor_Temperature:MAX31865xAP
- U5: symbol Regulator_Linear:AMS1117-3.3 -> Regulator_Linear:AP1117-15
- U6: footprint Package_DFN_QFN:QFN-24-1EP_4x4mm_P0.5mm_EP2.7x2.7mm -> Package_DFN_QFN:QFN-24-1EP_4x4mm_P0.5mm_EP2.6x2.6mm; symbol FW_Pumpengruppe:USB_UART_MIN -> Interface_USB:CP2102N-Axx-xQFN24
Connections:
- net RTD_RL_P is gone; now on net RTD_RL_FORCE_PLUS: U3.8 (FORCE+), X5.1 (Pin_1)
- net RTD_VL_P is gone; now on net RTD_VL_FORCE_PLUS: U2.8 (FORCE+), X4.1 (Pin_1)
- net +3V3: now also R21.1, R30.1, R31.1, U1.2 (VDD), U2.2 (DVDD), U2.3 (VDD), U3.2 (DVDD), U3.3 (VDD), U4.8 (VCC), U5.2 (VO), U6.5 (VIO), U6.6 (VDD), R33.2; no longer R21.2, R30.2, R31.2, U1.1 (GND), U1.15 (GND), U1.38 (GND), U1.39 (GND), U2.9 (SCK), U3.9 (SCK)
- net +5V: now also C60.2, C61.2, C62.2, C63.2, C64.2, C65.2, C66.2, C67.2, C68.2, C69.2, C70.2, C71.2, C72.2, C73.2, C74.2, C75.2, C76.2, C77.2, C78.2, C79.2, C80.2, C81.2, C82.2, C83.2, D20.2 (A), D21.2 (A), D60.2 (VSS), D61.2 (VSS), D62.2 (VSS), D63.2 (VSS), D64.2 (VSS), D65.2 (VSS), D66.2 (VSS), D67.2 (VSS), D68.2 (VSS), D69.2 (VSS), D70.2 (VSS), D71.2 (VSS), D72.2 (VSS), D73.2 (VSS), D74.2 (VSS), D75.2 (VSS), D76.2 (VSS), D77.2 (VSS), D78.2 (VSS), D79.2 (VSS), D80.2 (VSS), D81.2 (VSS), D82.2 (VSS), D83.2 (VSS), F2.2, K1.A1 (A1_5V), K2.A1 (A1_5V), K3.A1 (A1_5V), PSU1.3 (-Vout), Q1.2 (D), Q2.2 (D), Q3.2 (D), R1.2 (Pin_2), R10.1, R11.1, R12.1, R2.2 (Pin_2), R20.1, R32.2, R7.2, R8.2, R9.2, U1.1 (GND), U1.15 (GND), U1.38 (GND), U1.39 (GND), U2.13 (GND), U2.18 (DGND), U2.19 (GND), U3.13 (GND), U3.18 (DGND), U3.19 (GND), U4.5 (GND), U5.1 (GND), U5.3 (VI), U6.2 (GND), U6.25 (GND), X6.A1 (GND), X6.A12 (GND), X6.B1 (GND), X6.B12 (GND), X6.SH (SHIELD); no longer F2.1, K1.A2 (A2_DRV), K2.A2 (A2_DRV), K3.A2 (A2_DRV), R10.2, R11.2, R12.2, R20.2
- net BUS_5V: now also F2.1, J1.1 (Pin_1), J1.2 (Pin_2), J2.1 (Pin_1), J2.2 (Pin_2); no longer F2.2, J1.6 (Pin_6), J1.7 (Pin_7), J2.6 (Pin_6), J2.7 (Pin_7)
- net ESP_U0RX: now also D31.2 (A), U1.34 (RXD0/IO3), U6.21 (TXD); no longer U1.9 (IO33), U6.7 (DTR_NC)
- net ESP_U0TX: now also D30.2 (A), U1.35 (TXD0/IO1), U6.20 (RXD); no longer U1.7 (IO35), U6.6 (RXD_FROM_ESP_TX)
- net L_FUSED: now also F1.2, K1.1 (COM), K2.1 (COM), PSU1.1 (AC/L), R40.1, RV1.1; no longer F1.1, K1.2 (NO), K2.2 (NO), PSU1.2 (AC/N), R40.2, RV1.2
- net L_IN: now also F1.1, X1.1 (Pin_1); no longer F1.2, X1.3 (Pin_3)
- net L_PUMP: now also K1.2 (NO), X2.1 (Pin_1); no longer K1.1 (COM), X2.3 (Pin_3)
- net MIX_DIR_DRV: now also Q3.1 (G), R9.1; no longer U1.29 (IO5)
- net MIX_ENABLE_DRV: now also Q2.1 (G), R8.1; no longer U1.14 (IO12)
- net N: now also PSU1.2 (AC/N), RV1.2, X1.3 (Pin_3), X2.3 (Pin_3), X3.3 (Pin_3), X3.4 (Pin_4); no longer PSU1.1 (AC/L), RV1.1, X3.1 (Pin_1)
- net PUMP_DRV: now also Q1.1 (G), R7.1; no longer U1.16 (IO13)
- net RGB_DATA: now also U1.33 (IO21); no longer U1.27 (IO16)
- net RS485_A: now also D50.2 (A2), D51.1 (A1), D51.2 (A2), D52.2 (A2), J1.5 (Pin_5), J1.7 (Pin_7), J1.8 (Pin_8), J2.5 (Pin_5), J2.7 (Pin_7), J2.8 (Pin_8), J3.1 (Pin_1), J3.2 (Pin_2), J4.1 (Pin_1), J4.2 (Pin_2), JP1.2 (Pin_2), R32.1, U4.6 (A), U4.7 (B)
- net RS485_DE: now also U1.26 (IO4), U4.2 (~{RE}), U4.3 (DE); no longer U1.8 (IO32)
- net RS485_TERM: now also JP1.1 (Pin_1), R3.2 (Pin_2); no longer JP1.3 (Pin_3)
- net RS485_UART_RX: now also U1.27 (IO16), U4.1 (RO); no longer D31.2 (A), U1.33 (IO21)
- net RS485_UART_TX: now also U1.28 (IO17), U4.4 (DI); no longer D30.2 (A), U1.31 (IO19)
- net SPI_MISO: now also U1.31 (IO19), U2.17 (SDO), U3.17 (SDO); no longer U1.28 (IO17), U2.11 (MISO), U3.11 (MISO)
- net SPI_MOSI: now also U1.37 (IO23), U2.14 (SDI), U3.14 (SDI); no longer U1.13 (IO14)
- net SPI_SCK: now also U2.15 (SCLK), U3.15 (SCLK); no longer U2.16 (3V3), U3.16 (3V3)
- net USB_CC1: now also X6.A5 (CC1)
- net USB_CC2: now also X6.B5 (CC2)
- net USB_D+: now also U6.3 (D+), X6.A6 (D+), X6.B6 (D+); no longer X6.A7 (D-)
- net USB_D-: now also U6.4 (D-), X6.A7 (D-); no longer U6.3 (USB_D-), X6.A6 (D+)
- net USB_VBUS: now also U6.7 (VREGIN), U6.8 (VBUS), X6.A4 (VBUS), X6.A9 (VBUS), X6.B4 (VBUS), X6.B9 (VBUS); no longer U6.4 (GND), X6.B8 (SBU2)
- net RTD_VL_FORCE_PLUS: now reaches U2.10 (RTDIN+)
- net RTD_VL_FORCE_PLUS: now also U2.6 (REFIN-), U2.7 (ISENSOR), U2.9 (FORCE2), C22.1, R22.2
- net RTD_VL_FORCE_MINUS: now reaches X4.2 (Pin_2)
- net RTD_VL_FORCE_MINUS: now also U2.11 (RTDIN-), U2.12 (FORCE-), C22.2
- net RTD_RL_FORCE_PLUS: now reaches U3.10 (RTDIN+)
- net RTD_RL_FORCE_PLUS: now also U3.6 (REFIN-), U3.7 (ISENSOR), U3.9 (FORCE2), C23.1, R23.2
- net PUMP_DRV_GPIO: now reaches U1.10 (IO25)
- net PUMP_DRV_GPIO: now also R4.1
- net MIX_ENABLE_DRV_GPIO: now reaches U1.11 (IO26)
- net MIX_ENABLE_DRV_GPIO: now also R5.1
- net MIX_DIR_DRV_GPIO: now reaches U1.12 (IO27)
- net MIX_DIR_DRV_GPIO: now also R6.1
- net ESP_EN: now reaches U1.3 (EN)
- net ESP_EN: now also R33.1
- net RTD_RL_CS: now reaches U1.36 (IO22)
- net RTD_RL_CS: now also U3.16 (~{CS})
- net RTD_RL_FORCE_MINUS: now reaches X5.2 (Pin_2)
- net RTD_RL_FORCE_MINUS: now also U3.11 (RTDIN-), U3.12 (FORCE-), C23.2
- removed net GND: C60.2, C61.2, C62.2, C63.2, C64.2, C65.2, C66.2, C67.2, C68.2, C69.2, C70.2, C71.2, C72.2, C73.2, C74.2, C75.2, C76.2, C77.2, C78.2, C79.2, C80.2, C81.2, C82.2, C83.2, D20.2 (A), D21.2 (A), D60.2 (VSS), D61.2 (VSS), D62.2 (VSS), D63.2 (VSS), D64.2 (VSS), D65.2 (VSS), D66.2 (VSS), D67.2 (VSS), D68.2 (VSS), D69.2 (VSS), D70.2 (VSS), D71.2 (VSS), D72.2 (VSS), D73.2 (VSS), D74.2 (VSS), D75.2 (VSS), D76.2 (VSS), D77.2 (VSS), D78.2 (VSS), D79.2 (VSS), D80.2 (VSS), D81.2 (VSS), D82.2 (VSS), D83.2 (VSS), PSU1.3 (-Vout), Q1.3 (S), Q2.3 (S), Q3.3 (S), R32.1, R7.1, R8.1, R9.1, U1.2 (VDD), U2.1 (RTD+), U3.1 (RTD+), U6.1 (VBUS), X6.A4 (VBUS), X6.A9 (VBUS), X6.B4 (VBUS), X6.B9 (VBUS)
- net LED230_A renamed MAINS_LED_K
- net MAINS_LED_K: now also R41.2; no longer R41.1
- removed net LED230_DROP: R40.1, R41.2
- net LED_3V3_A renamed LED_3V3_K
- net LED_3V3_K: now also R21.2; no longer R21.1
- net LED_5V_A renamed LED_5V_K
- net LED_5V_K: now also R20.2; no longer R20.1
- net LED_CLOSE_A renamed LED_MIX_DIR_K
- net LED_MIX_DIR_K: now also R12.2; no longer R12.1
- net LED_OPEN_A renamed LED_MIX_ENABLE_K
- net LED_MIX_ENABLE_K: now also R11.2; no longer R11.1
- net LED_PUMP_A renamed LED_PUMP_K
- net LED_PUMP_K: now also R10.2; no longer R10.1
- net LED_RX_A renamed LED_USB_RX_K
- net LED_USB_RX_K: now also R31.2; no longer R31.1
- net LED_TX_A renamed LED_USB_TX_K
- net LED_USB_TX_K: now also R30.2; no longer R30.1
- net L_CLOSE renamed L_MIX_CLOSE
- net L_OPEN renamed L_MIX_ENABLE
- net L_MIX_ENABLE: now also K2.2 (NO); no longer X3.3 (Pin_3)
- net MIX_DIR_COIL_L renamed MIX_DIR_COIL_DRV
- net MIX_DIR_COIL_DRV: now also K3.A2 (A2_DRV), Q3.3 (S); no longer K3.A1 (A1_5V), Q3.2 (D)
- removed net MIX_DIR_GATE: Q3.1 (G), R6.1, R9.2
- net MIX_ENABLE_COIL_L renamed MIX_ENABLE_COIL_DRV
- net MIX_ENABLE_COIL_DRV: now also K2.A2 (A2_DRV), Q2.3 (S); no longer K2.A1 (A1_5V), Q2.2 (D)
- removed net MIX_ENABLE_GATE: Q2.1 (G), R5.1, R8.2
- net MIX_L_EN renamed L_MIX_OPEN
- net L_MIX_OPEN: now also X3.1 (Pin_1); no longer K2.1 (COM)
- removed net PE: X1.1 (Pin_1), X2.1 (Pin_1)
- net PUMP_COIL_L renamed PUMP_COIL_DRV
- net PUMP_COIL_DRV: now also K1.A2 (A2_DRV), Q1.3 (S); no longer K1.A1 (A1_5V), Q1.2 (D)
- removed net PUMP_GATE: Q1.1 (G), R4.1, R7.2
- net RGB_DIN_1 renamed RGB_D60_DIN
- net RGB_DOUT_1 renamed RGB_D60_DOUT
- net RGB_DOUT_10 renamed RGB_D69_DOUT
- net RGB_DOUT_11 renamed RGB_D70_DOUT
- net RGB_DOUT_12 renamed RGB_D71_DOUT
- net RGB_DOUT_13 renamed RGB_D72_DOUT
- net RGB_DOUT_14 renamed RGB_D73_DOUT
- net RGB_DOUT_15 renamed RGB_D74_DOUT
- net RGB_DOUT_16 renamed RGB_D75_DOUT
- net RGB_DOUT_17 renamed RGB_D76_DOUT
- net RGB_DOUT_18 renamed RGB_D77_DOUT
- net RGB_DOUT_19 renamed RGB_D78_DOUT
- net RGB_DOUT_2 renamed RGB_D61_DOUT
- net RGB_DOUT_20 renamed RGB_D79_DOUT
- net RGB_DOUT_21 renamed RGB_D80_DOUT
- net RGB_DOUT_22 renamed RGB_D81_DOUT
- net RGB_DOUT_23 renamed RGB_D82_DOUT
- net RGB_DOUT_3 renamed RGB_D62_DOUT
- net RGB_DOUT_4 renamed RGB_D63_DOUT
- net RGB_DOUT_5 renamed RGB_D64_DOUT
- net RGB_DOUT_6 renamed RGB_D65_DOUT
- net RGB_DOUT_7 renamed RGB_D66_DOUT
- net RGB_DOUT_8 renamed RGB_D67_DOUT
- net RGB_DOUT_9 renamed RGB_D68_DOUT
- removed net RS485_B: D51.1 (A1), D52.2 (A2), J1.3 (Pin_3), J2.3 (Pin_3), J3.2 (Pin_2), J4.2 (Pin_2), JP1.2 (Pin_2)
- removed net RS485_GND: D50.2 (A2), D51.2 (A2), J1.1 (Pin_1), J2.1 (Pin_1), J3.1 (Pin_1), J4.1 (Pin_1), R32.2
- new net MAINS_LED_SERIES: R40.2, R41.1
- new net RTD_RL_BIAS: R23.1, U3.4 (BIAS), U3.5 (REFIN+)
- new net RTD_VL_BIAS: R22.1, U2.4 (BIAS), U2.5 (REFIN+)
- new net RTD_VL_CS: U1.29 (IO5), U2.16 (~{CS})
- no-connect marks 25 -> 46
Other:
- moved on the sheet: C60, C61, C62, C63, D41, D60, D61, D62, D63, F1, J1, J2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

Commit message: sicherung
Parts:
- removed U6: CP2102N-A02-GQFN24, Package_DFN_QFN:QFN-24-1EP_4x4mm_P0.5mm_EP2.6x2.6mm, symbol Interface_USB:CP2102N-Axx-xQFN24
- added H1, H2, H3, H4: MountingHole_M3, MountingHole:MountingHole_3.2mm_M3, symbol Mechanical:MountingHole
- added J5: EXT_GPIO_HEADER, Connector_PinHeader_2.54mm:PinHeader_2x10_P2.54mm_Vertical, symbol Connector_Generic:Conn_02x10_Odd_Even
- added R90: 10k 1% 0603, Resistor_SMD:R_0603_1608Metric, symbol Device:R
- added SW1: BOOT/CFG RESET, Button_Switch_SMD:SW_Push_1TS009xxxx-xxxx-xxxx_6x6x5mm, symbol Switch:SW_Push
- J3, J4: value 3-pin 3.5mm terminal -> KF128L-3.5-3P; footprint FW_Pumpengruppe:TB_3_350 -> FW_Pumpengruppe:TB_KF128L_350_3P; AISLER_MPN DG350-3.5-03P-14-00AH -> KF128L-3.5-3P; MPN DG350-3.5-03P-14-00AH -> KF128L-3.5-3P; Manufacturer Degson -> Cixi Kefa Elec
- K1: value G5LE-1A-E DC5 -> SRD-05VDC-SL-C; footprint FW_Pumpengruppe:Relay_SPST_16A -> Relay_THT:Relay_SPDT_SANYOU_SRD_Series_Form_C; AISLER_MPN G5LE-1A-E DC5 -> SRD-05VDC-SL-C; AssemblyNote VERIFY_FOOTPRINT before assembly, relay footprint is still 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 -> Costdown SRD Form-C relay; K1/K2 NC contact intentionally u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; MPN G5LE-1A-E DC5 -> SRD-05VDC-SL-C; Manufacturer Omron -> Songle Relay; now in the parts list
- K2: value G5LE-1A-E DC5 -> SRD-05VDC-SL-C; footprint FW_Pumpengruppe:Relay_SPST_8A -> Relay_THT:Relay_SPDT_SANYOU_SRD_Series_Form_C; AISLER_MPN G5LE-1A-E DC5 -> SRD-05VDC-SL-C; AssemblyNote VERIFY_FOOTPRINT before assembly, relay footprint is still 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 -> Costdown SRD Form-C relay; K1/K2 NC contact intentionally u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; MPN G5LE-1A-E DC5 -> SRD-05VDC-SL-C; Manufacturer Omron -> Songle Relay
- K3: value G5LE-1 DC5 -> SRD-05VDC-SL-C; footprint FW_Pumpengruppe:Relay_SPDT_8A -> Relay_THT:Relay_SPDT_SANYOU_SRD_Series_Form_C; AISLER_MPN G5LE-1 DC5 -> SRD-05VDC-SL-C; AssemblyNote VERIFY_FOOTPRINT before assembly, relay footprint is still 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 -> Costdown SRD Form-C relay; K1/K2 NC contact intentionally u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; MPN G5LE-1 DC5 -> SRD-05VDC-SL-C; Manufacturer Omron -> Songle Relay
- PSU1: value IRM-05-5 -> HLK-5M05; footprint Converter_ACDC:Converter_ACDC_MeanWell_IRM-05-xx_THT -> Converter_ACDC:Converter_ACDC_Hi-Link_HLK-5Mxx; AISLER_MPN IRM-05-5 -> HLK-5M05; AssemblyNote AISLER assembly target PSU; verify 230VAC clearance and fin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 -> 5W AC/DC module; re-route mains and SELV clearances after f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; MPN IRM-05-5 -> HLK-5M05; Manufacturer Mean Well -> Hi-Link
- U1: value ESP32-WROOM-32D-N4 -> ESP32-S3-WROOM-1-N4; footprint RF_Module:ESP32-WROOM-32D -> RF_Module:ESP32-S3-WROOM-1; symbol RF_Module:ESP32-WROOM-32 -> RF_Module:ESP32-S3-WROOM-1; AISLER_MPN ESP32-WROOM-32D-N4 -> ESP32-S3-WROOM-1-N4; MPN ESP32-WROOM-32D-N4 -> ESP32-S3-WROOM-1-N4; Supplier AISLER source or equivalent -> LCSC or PCBWay equivalent
- X1, X2: value 3-pin 7.62mm terminal -> KF128-5.08-3P-AA; footprint FW_Pumpengruppe:TB_3_762 -> FW_Pumpengruppe:TB_KF128_508_3P; AISLER_MPN DG129-7.62-03P-14-00AH -> KF128-5.08-3P-AA; MPN DG129-7.62-03P-14-00AH -> KF128-5.08-3P-AA; Manufacturer Degson -> Cixi Kefa Elec
- X3: value 4-pin 7.62mm terminal -> DB128L-5.08-4P-GN-S; footprint FW_Pumpengruppe:TB_4_762 -> FW_Pumpengruppe:TB_DB128L_508_4P; AISLER_MPN DG129-7.62-04P-14-00AH -> DB128L-5.08-4P-GN-S; MPN DG129-7.62-04P-14-00AH -> DB128L-5.08-4P-GN-S; Manufacturer Degson -> DORABO
- X4, X5: value 2-pin 3.5mm terminal -> KF128L-3.5-2P; footprint FW_Pumpengruppe:TB_2_350 -> FW_Pumpengruppe:TB_KF128L_350_2P; AISLER_MPN DG350-3.5-02P-14-00AH -> KF128L-3.5-2P; MPN DG350-3.5-02P-14-00AH -> KF128L-3.5-2P; Manufacturer Degson -> Cixi Kefa Elec
Connections:
- net +3V3: now also R33.1, J5.3 (Pin_3), R90.2; no longer R33.2
- net +5V: now also U1.40 (GND), U1.41 (GND), J5.1 (Pin_1), J5.2 (Pin_2), J5.20 (Pin_20), J5.4 (Pin_4), SW1.2; no longer U1.15 (GND), U1.38 (GND), U1.39 (GND)
- net ESP_EN: now also R33.2; no longer R33.1
- net ESP_U0RX: no longer U1.34 (RXD0/IO3)
- net ESP_U0TX: no longer U1.35 (TXD0/IO1)
- net MIX_DIR_DRV_GPIO: now also U1.30 (IO37); no longer U1.12 (IO27)
- net MIX_ENABLE_DRV_GPIO: now also U1.29 (IO36); no longer U1.11 (IO26)
- net PUMP_DRV_GPIO: now also U1.28 (IO35); no longer U1.10 (IO25)
- net RGB_DATA: now also U1.23 (IO21); no longer U1.33 (IO21)
- net RS485_DE: now also U1.4 (IO4); no longer U1.26 (IO4)
- net RS485_UART_RX: now also U1.9 (IO16); no longer U1.27 (IO16)
- net RS485_UART_TX: now also U1.10 (IO17); no longer U1.28 (IO17)
- net RTD_RL_CS: now also U1.17 (IO9); no longer U1.36 (IO22)
- net RTD_VL_CS: now also U1.18 (IO10); no longer U1.29 (IO5)
- net SPI_MISO: now also U1.21 (IO13); no longer U1.31 (IO19)
- net SPI_MOSI: now also U1.19 (IO11); no longer U1.37 (IO23)
- net SPI_SCK: now also U1.20 (IO12); no longer U1.30 (IO18)
- net USB_D+: now also U1.14 (USB_D+)
- net USB_D-: now also U1.13 (USB_D-)
- net ESP_IO46_EXT: now reaches U1.16 (IO46)
- net ESP_IO14_EXT: now reaches U1.22 (IO14)
- net ESP_IO14_EXT: now also J5.12 (Pin_12)
- net ESP_IO47_EXT: now reaches U1.24 (IO47)
- net ESP_IO48_EXT: now reaches U1.25 (IO48)
- net ESP_IO39_EXT: now reaches U1.32 (IO39)
- net ESP_IO39_EXT: now also J5.16 (Pin_16)
- net ESP_IO5_EXT: now reaches U1.5 (IO5)
- net ESP_IO5_EXT: now also J5.8 (Pin_8)
- net ESP_IO6_EXT: now reaches U1.6 (IO6)
- net ESP_IO6_EXT: now also J5.9 (Pin_9)
- net ESP_IO7_EXT: now reaches U1.7 (IO7)
- net ESP_IO7_EXT: now also J5.10 (Pin_10)
- net ESP_IO15_EXT: now reaches U1.8 (IO15)
- net ESP_IO15_EXT: now also J5.13 (Pin_13)
- new net ESP_IO0_BOOT: R90.1, SW1.1, U1.27 (IO0)
- new net ESP_IO18_EXT: J5.14 (Pin_14), U1.11 (IO18)
- new net ESP_IO1_EXT: J5.5 (Pin_5), U1.39 (IO1)
- new net ESP_IO2_EXT: J5.6 (Pin_6), U1.38 (IO2)
- new net ESP_IO38_EXT: J5.15 (Pin_15), U1.31 (IO38)
- new net ESP_IO3_EXT: J5.7 (Pin_7), U1.15 (IO3)
- new net ESP_IO40_EXT: J5.17 (Pin_17), U1.33 (IO40)
- new net ESP_IO41_EXT: J5.18 (Pin_18), U1.34 (IO41)
- new net ESP_IO42_EXT: J5.19 (Pin_19), U1.35 (IO42)
- new net ESP_IO45_EXT: U1.26 (IO45)
- new net ESP_IO8_EXT: J5.11 (Pin_11), U1.12 (IO8)
- new net ESP_RXD0_EXT: U1.36 (RXD0)
- new net ESP_TXD0_EXT: U1.37 (TXD0)
- no-connect marks 46 -> 28
Other:
- note added: "SELV / CONTROL ZONE - U1: ESP32-WROOM-32D, PCB-Antenne am Platinenrand/Keepout - X6: USB-C direkt an ESP32-S3 Native-USB fuer Firmware/Debug - U2/U3: MAX31865 RTD VL/RL - U4: MAX3485/SP3485 RS485-Standardtransceiver, DE/RE per RS485_DE - J1/J2 RJ45 + J3/J4 Schraubklemmen liegen parallel - WLAN nur Konfiguration/OTA, Regelbetrieb ueber Modbus RTU"
- note added: "SELV-/MCU-LOGIK PSU1 HLK-5M05 5V -> U5 -> 3V3 U1 ESP32-S3-WROOM-1-N4: PCB-Antenne am Platinenrand/Keepout U1 ESP32-S3: native USB, feste GPIOs fuer Relais/RS485/SPI/RGB; J5 fuehrt freie GPIOs + 5V/3V3/GND heraus Treiber je Relais: 100R Gate, 100k Pulldown, AO3400A, SS14 Freilauf, Status-LED U2/U3 MAX31865: SPI auf festen S3-GPIOs, je Sensor eigener CS X4 RTD_VL_P/N, X5 RTD_RL_P/N"
- note removed: "SELV / CONTROL ZONE - U1: ESP32-WROOM-32D, PCB-Antenne am Platinenrand/Keepout - X6/U6: USB-C Service + USB-UART fuer Firmware/Debug - U2/U3: MAX31865 RTD VL/RL - U4: MAX3485/SP3485 RS485-Standardtransceiver, DE/RE per RS485_DE - J1/J2 RJ45 + J3/J4 Schraubklemmen liegen parallel - WLAN nur Konfiguration/OTA, Regelbetrieb ueber Modbus RTU"
- note removed: "SELV-/MCU-LOGIK PSU1 IRM-05-5 5V -> U5 -> 3V3 U1 ESP32-WROOM-32D: PCB-Antenne am Platinenrand/Keepout U1 GPIO25/26/27 -> NMOS-Treiber: PUMP_DRV, MIX_ENABLE_DRV, MIX_DIR_DRV; GPIO4=RS485_DE Treiber je Relais: 100R Gate, 100k Pulldown, AO3400A, SS14 Freilauf, Status-LED U2/U3 MAX31865: VSPI GPIO23=MOSI, GPIO19=MISO, GPIO18=SCK X4 RTD_VL_P/N, X5 RTD_RL_P/N"

Commit message: sicherung
Parts:
- F1: value 5x20 fuse holder -> 2x FC-203-22 fuse clips for 5x20; footprint FW_Pumpengruppe:FUSE_5X20 -> Fuse:Fuseholder_Clip-5x20mm_Bel_FC-203-22_Lateral_P17.80x5.00mm_D1.17mm_Horizontal; AISLER_MPN 03453LS1H -> FC-203-22; AssemblyNote 5x20 PCB fuse holder/fuse solution, verify footprint and fu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 -> Populate two FC-203-22 clips per F1 footprint for one 5x20m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; MPN 03453LS1H -> FC-203-22; Manufacturer Littelfuse -> Bel Fuse; Supplier AISLER source or equivalent -> LCSC C3205463 / PCBWay equivalent
- J3: Supplier AISLER source or equivalent -> LCSC C474931 / PCBWay equivalent
- K1, K2, K3: Supplier AISLER source or equivalent -> LCSC C35449 / PCBWay equivalent
- U4: value MAX3485EESA+ -> SP3485EN-L/TR; AISLER_MPN MAX3485EESA+ -> SP3485EN-L/TR; MPN MAX3485EESA+ -> SP3485EN-L/TR; Manufacturer Analog Devices -> MaxLinear; Supplier AISLER source or equivalent -> LCSC C8963 / PCBWay equivalent
Changed lines of the file:
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@@
 			)
 		)
-		(property "Supplier" "AISLER source or equivalent"
+		(property "Supplier" "LCSC C35449 / PCBWay equivalent"
 			(at 386.08 -147.32 0
 			)
@@
 			)
 		)
-		(property "Supplier" "AISLER source or equivalent"
+		(property "Supplier" "LCSC C474931 / PCBWay equivalent"
 			(at 220 142 0
 			)
@@
 			)
 		)
-		(property "Value" "MAX3485EESA+"
+		(property "Value" "SP3485EN-L/TR"
 			(at 728.08 -51.13 0
 			)
@@
 			)
 		)
-		(property "Manufacturer" "Analog Devices"
+		(property "Manufacturer" "MaxLinear"
 			(at 728.08 -62.13 0
 			)
@@
 			)
 		)
-		(property "MPN" "MAX3485EESA+"
+		(property "MPN" "SP3485EN-L/TR"
 			(at 728.08 -62.13 0
 			)
@@
 			)
 		)
-		(property "Supplier" "AISLER source or equivalent"
+		(property "Supplier" "LCSC C8963 / PCBWay equivalent"
 			(at 728.08 -62.13 0
 			)
@@
 			)
 		)
-		(property "AISLER_MPN" "MAX3485EESA+"
+		(property "AISLER_MPN" "SP3485EN-L/TR"
 			(at 728.08 -62.13 0
 			)
@@
 			)
 		)
-		(property "Supplier" "AISLER source or equivalent"
+		(property "Supplier" "LCSC C35449 / PCBWay equivalent"
 			(at 541.02 -176.53 0
 			)
@@
 			)
 		)
-		(property "Value" "5x20 fuse holder"
+		(property "Value" "2x FC-203-22 fuse clips for 5x20"
 			(at 2.54 45.37 0
 			)
@@
 			)
 		)
-		(property "Footprint" "FW_Pumpengruppe:FUSE_5X20"
+		(property "Footprint" "Fuse:Fuseholder_Clip-5x20mm_Bel_FC-203-22_Lateral_P17.80x5.00mm_D1.17mm_Horizontal"
 			(at 2.54 49.37 0
 			)
@@
 			)
 		)
-		(property "Manufacturer" "Littelfuse"
+		(property "Manufacturer" "Bel Fuse"
 			(at 2.54 39.37 0
 			)
@@
 			)
 		)
-		(property "MPN" "03453LS1H"
+		(property "MPN" "FC-203-22"
 			(at 2.54 39.37 0
 			)
@@
 			)
 		)
-		(property "Supplier" "AISLER source or equivalent"
+		(property "Supplier" "LCSC C3205463 / PCBWay equivalent"
 			(at 2.54 39.37 0
 			)
@@
 			)
 		)
-		(property "AssemblyNote" "5x20 PCB fuse holder/fuse solution, verify footprint and fuse rating before order"
+		(property "AssemblyNote" "Populate two FC-203-22 clips per F1 footprint for one 5x20mm fuse; do not use one-piece expensive fuse holder"
 			(at 2.54 39.37 0
 			)
@@
 			)
 		)
-		(property "AISLER_MPN" "03453LS1H"
+		(property "AISLER_MPN" "FC-203-22"
 			(at 2.54 39.37 0
 			)
@@
 			)
 		)
-		(property "Supplier" "AISLER source or equivalent"
+		(property "Supplier" "LCSC C35449 / PCBWay equivalent"
 			(at 459.74 -161.29 0
 			)

Commit message: sicherung
Parts:
- R90: Manufacturer (none) -> Yageo
- SW1: Manufacturer (none) -> HYP / equivalent
Changed lines of the file:
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@@
 		(property "Footprint" "Button_Switch_SMD:SW_Push_1TS009xxxx-xxxx-xxxx_6x6x5mm" (at 700 15.08 0) (hide yes) (effects (font (size 1.27 1.27))))
 		(property "MPN" "1TS009A-1800-5000-CT" (at 700 10 0) (hide yes) (effects (font (size 1.27 1.27))))
+		(property "Manufacturer" "HYP / equivalent" (at 700 12 0) (hide yes) (effects (font (size 1.27 1.27))))
 		(pin "1")
 		(pin "2")
@@
 		(property "Footprint" "Resistor_SMD:R_0603_1608Metric" (at 700 -1.778 0) (hide yes) (effects (font (size 1.27 1.27))))
 		(property "MPN" "RC0603FR-0710KL" (at 700 0 90) (hide yes) (effects (font (size 1.27 1.27))))
+		(property "Manufacturer" "Yageo" (at 700 0 90) (hide yes) (effects (font (size 1.27 1.27))))
 		(pin "1")
 		(pin "2")
